File: Annahs_clock_hps/Annahs_clock_hps.kicad_sch (KiCad schematic)
At the start: 55 parts, among them J1 Conn_01x06, J2 Power_inlet_vertical, J3 Conn_02x03_Odd_Even, SW1 Omron_B3F_SPST, SW2 Omron_B3F_SPST, SW3 Omron_B3F_SPST, SW4 Omron_B3F_SPST, SW5 Omron_B3F_SPST, SW6 Omron_B3F_SPST, U1 DS1307_DIP-8, U2 MAX7219, U3 L7805, U4 SC56-11EWA, U5 SC56-11EWA, Y1 Crystal_16MHz, Y2 Crystal_32768Hz

Commit message: Updated Schematic
Connections:
- net GND: now also RV1.1; no longer RV1.3
- net VCC: now also RV1.3; no longer RV1.1
Changed lines of the file:
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@@
     (pin "1")
   )
-  (symbol (lib_id "HPS:GND") (at 278.13 138.43 180) (unit 1)
-    (in_bom yes) (on_board yes) (fields_autoplaced)
-    (property "Reference" "#PWR036" (id 0) (at 278.13 132.08 0)
-      (effects (font (size 1.27 1.27)) hide)
-    )
-    (property "Value" "GND" (id 1) (at 278.13 133.35 0))
-    (property "Footprint" "" (id 2) (at 278.13 138.43 0)
-      (effects (font (size 1.27 1.27)) hide)
-    )
-    (property "Datasheet" "" (id 3) (at 278.13 138.43 0)
+  (symbol (lib_id "HPS:GND") (at 278.13 146.05 0) (unit 1)
+    (in_bom yes) (on_board yes) (fields_autoplaced)
+    (property "Reference" "#PWR036" (id 0) (at 278.13 152.4 0)
+      (effects (font (size 1.27 1.27)) hide)
+    )
+    (property "Value" "GND" (id 1) (at 278.13 151.13 0))
+    (property "Footprint" "" (id 2) (at 278.13 146.05 0)
+      (effects (font (size 1.27 1.27)) hide)
+    )
+    (property "Datasheet" "" (id 3) (at 278.13 146.05 0)
       (effects (font (size 1.27 1.27)) hide)
     )
@@
     )
   )
-  (symbol (lib_id "HPS:VCC") (at 278.13 146.05 180) (unit 1)
+  (symbol (lib_id "HPS:VCC") (at 278.13 138.43 0) (unit 1)
     (in_bom yes) (on_board yes) (fields_autoplaced)
     (property "Reference" "#PWR037" (id 0) (at 278.13 142.24 0)
       (effects (font (size 1.27 1.27)) hide)
     )
-    (property "Value" "VCC" (id 1) (at 278.13 151.13 0))
-    (property "Footprint" "" (id 2) (at 278.13 146.05 0)
-      (effects (font (size 1.27 1.27)) hide)
-    )
-    (property "Datasheet" "" (id 3) (at 278.13 146.05 0)
-      (effects (font (size 1.27 1.27)) hide)
-    )
+    (property "Value" "VCC" (id 1) (at 278.13 133.35 0))
+    (property "Footprint" "" (id 2) (at 278.13 138.43 0)
+      (effects (font (size 1.27 1.27)) hide)
+    )
+    (property "Datasheet" "" (id 3) (at 278.13 138.43 0)
+      (effects (font (size 1.27 1.27)) hide)
+    )

Commit message: PCB and Schematic Updated
Parts:
- removed H1, H2, H3, H4: MountingHole, footprints:MountingHole_3.2mm_M3, symbol HPS:MountingHole
- removed R12, R13, R14, R15: R_0805_10K, footprints:R_0805_2012Metric, symbol HPS:R_0805_10K
- added R12, R13, R14, R15: R_0805_1K, footprints:R_0805_2012Metric, symbol HPS:R_0805_1K
- added R17: R_0805_47, footprints:R_0805_2012Metric, symbol HPS:R_0805_47
Connections:
- net Alarm_SW: now also R14.1
- net Down_SW: now also R12.1
- net GND: now also R16.1, R16.2
- net Select_SW: now also R13.1
- net Up_SW: now also R15.1
- net VCC: now also R17.2; no longer R16.1
- net at R9.1, SW4.3 (B), SW4.4 (B): now also R15.2
- net at R1.1, SW2.3 (B), SW2.4 (B): now also R12.2
- net at DS1.15 (LED(+)): now also R17.1; no longer R16.2
- net at R8.1, SW3.3 (B), SW3.4 (B): now also R14.2
- net at R2.1, SW1.3 (B), SW1.4 (B): now also R13.2
Other:
- note removed: "Mechanical"
- moved on the sheet: R16

Commit message: Updated Schematic and PCB
Parts:
- removed C12: C_0805_0.1uf, footprints:C_0805_2012Metric, symbol HPS:C_0805_0.1uf
- removed R14: R_0805_1K, footprints:R_0805_2012Metric, symbol HPS:R_0805_1K
- added Q1: NPN_2N3904_SOT23, footprints:SOT-23, symbol HPS:NPN_2N3904_SOT23
- added R14: R_0805_2.2K, footprints:R_0805_2012Metric, symbol HPS:R_0805_2.2K
- U3: Digikey PN (none) -> 497-7255-1-ND; MFG (none) -> STMicroelectronics; MPN (none) -> L7805CDT-TR
Connections:
- net GND: now also Q1.2 (E); no longer BZ1.2 (+), R16.1
- net MISO: now also R8.1, SW3.3 (B), SW3.4 (B); no longer BZ1.1 (-)
- net VCC: now also BZ1.2 (+)
- net at DS1.16 (LED(-)), SW6.3 (B), SW6.4 (B): now also R16.1
- net Alarm_SW renamed Buzzer
- net Buzzer: now also R14.1
- new net: Q1.1 (B), R14.2
- new net: BZ1.1 (-), Q1.3 (C)
Other:
- moved on the sheet: BZ1, C13, C8, C9, R10, R15, R8, R9, SW3, SW4

Commit message: Schematic and PCB Updates
Parts:
- added TP1, TP10, TP11, TP12, TP13, TP14, TP2, TP3, TP4, TP5, TP6, TP7, TP8, TP9: TestPoint, footprints:TestPoint_THTPad_D2.0mm_Drill1.0mm, symbol HPS:TestPoint
Connections:
- net Dig01_A: now also TP3.1
- net Dig01_B: now also TP4.1
- net Dig01_C: now also TP5.1
- net Dig01_D: now also TP6.1
- net Dig01_DP: now also TP10.1
- net Dig01_E: now also TP7.1
- net Dig01_F: now also TP8.1
- net Dig01_G: now also TP9.1
- net Dig0_Com: now also TP11.1
- net Dig1_Com: now also TP1.1
- net GND: now also BZ1.2 (+), D1.1 (K), Q1.3 (C), TP12.1, TP13.1; no longer R11.2
- net LED_SCK: now also R11.1; no longer D1.2 (A)
- net VCC: now also BZ1.1 (-), TP14.1, TP2.1; no longer BZ1.2 (+)
- new net: D1.2 (A), R11.2
Other:
- note added: "Power TP"
- moved on the sheet: D1, R11
