File: Annahs_clock_hps/Annahs_clock_hps.kicad_sch (KiCad schematic)
At the start: 73 parts, among them J1 Conn_01x06, J2 Power_inlet_vertical, J3 Conn_02x03_Odd_Even, Q1 NPN_2N3904_SOT23, SW1 Omron_B3F_SPST, SW2 Omron_B3F_SPST, SW3 Omron_B3F_SPST, SW4 Omron_B3F_SPST, SW5 Omron_B3F_SPST, SW6 Omron_B3F_SPST, U1 DS1307_DIP-8, U2 MAX7219, U3 L7805, U4 SC56-11EWA, U5 SC56-11EWA, Y1 Crystal_16MHz, Y2 Crystal_32768Hz

Commit message: Updated Schematic and PCB
Parts:
- added TP17, TP18, TP19: TestPoint, footprints:TestPoint_THTPad_D2.0mm_Drill1.0mm, symbol HPS:TestPoint
Connections:
- net LED_SCK: now also TP17.1
- net MAX_Load: now also TP18.1
- net MOSI: now also TP19.1
Changed lines of the file:
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@@
   (junction (at 290.83 64.77) (diameter 0) (color 0 0 0 0)
   )
+  (junction (at 237.49 82.55) (diameter 0) (color 0 0 0 0)
+  )
   (junction (at 266.7 191.77) (diameter 0) (color 0 0 0 0)
   )
@@
   (junction (at 152.4 248.92) (diameter 0) (color 0 0 0 0)
   )
+  (junction (at 212.09 85.09) (diameter 0) (color 0 0 0 0)
+  )
   (junction (at 356.87 29.21) (diameter 0) (color 0 0 0 0)
   )
@@
   (junction (at 387.35 77.47) (diameter 0) (color 0 0 0 0)
   )
+  (junction (at 237.49 87.63) (diameter 0) (color 0 0 0 0)
+  )
   (junction (at 87.63 171.45) (diameter 0) (color 0 0 0 0)
   )
@@
     (stroke (width 0) (type default) (color 0 0 0 0))
   )
+  (wire (pts (xy 237.49 87.63) (xy 240.03 87.63))
+    (stroke (width 0) (type default) (color 0 0 0 0))
+  )
   (polyline (pts (xy 350.52 198.12) (xy 350.52 203.2))
     (stroke (width 0) (type default) (color 0 0 0 0))
@@
     (stroke (width 0) (type default) (color 0 0 0 0))
   )
+  (wire (pts (xy 237.49 82.55) (xy 240.03 82.55))
+    (stroke (width 0) (type default) (color 0 0 0 0))
+  )
   (wire (pts (xy 273.05 67.31) (xy 260.35 67.31))
     (stroke (width 0) (type default) (color 0 0 0 0))
@@
     (stroke (width 0) (type default) (color 0 0 0 0))
   )
-  (wire (pts (xy 222.25 85.09) (xy 240.03 85.09))
+  (wire (pts (xy 209.55 85.09) (xy 212.09 85.09))
     (stroke (width 0) (type default) (color 0 0 0 0))
   )
@@
     (stroke (width 0) (type default) (color 0 0 0 0))
   )
-  (wire (pts (xy 234.95 82.55) (xy 240.03 82.55))
+  (wire (pts (xy 234.95 82.55) (xy 237.49 82.55))
     (stroke (width 0) (type default) (color 0 0 0 0))
   )
@@
     (stroke (width 0) (type default) (color 0 0 0 0))
   )
-  (wire (pts (xy 233.68 87.63) (xy 240.03 87.63))
+  (wire (pts (xy 233.68 87.63) (xy 237.49 87.63))
     (stroke (width 0) (type default) (color 0 0 0 0))
   )
@@
     (stroke (width 0) (type default) (color 0 0 0 0))
   )
+  (wire (pts (xy 212.09 85.09) (xy 240.03 85.09))
+    (stroke (width 0) (type default) (color 0 0 0 0))
+  )
   (wire (pts (xy 356.87 64.77) (xy 356.87 29.21))
     (stroke (width 0) (type default) (color 0 0 0 0))
@@
     )
   )
-  (global_label "LED_SCK" (shape input) (at 222.25 85.09 180) (fields_autoplaced)
+  (global_label "LED_SCK" (shape input) (at 209.55 85.09 180) (fields_autoplaced)
     (effects (font (size 1.27 1.27)) (justify right))
-    (property "Intersheet References" "${INTERSHEET_REFS}" (id 0) (at 211.6726 85.0106 0)
+    (property "Intersheet References" "${INTERSHEET_REFS}" (id 0) (at 198.9726 85.0106 0)
       (effects (font (size 1.27 1.27)) (justify right) hide)
     )
@@
     (pin "1")
   )
+  (symbol (lib_id "HPS:TestPoint") (at 212.09 85.09 0) (unit 1)
+    (in_bom yes) (on_board yes)
+    (property "Reference" "TP17" (id 0) (at 209.55 76.2 0)
+      (effects (font (size 1.27 1.27)) (justify left))
+    )
+    (property "Value" "TestPoint" (id 1) (at 209.55 78.74 0)
+      (effects (font (size 1.27 1.27)) (justify left))
+    )
+    (property "Footprint" "footprints:TestPoint_THTPad_D2.0mm_Drill1.0mm" (id 2) (at 217.17 85.09 0)
+      (effects (font (size 1.27 1.27)) hide)
+    )
+    (property "Datasheet" "~" (id 3) (at 217.17 85.09 0)
+      (effects (font (size 1.27 1.27)) hide)
+    )
+    (pin "1")
+  )
   (symbol (lib_id "HPS:Crystal_32768Hz") (at 276.86 198.12 270) (unit 1)
     (in_bom yes) (on_board yes)
@@
   (symbol (lib_id "HPS:C_0805_10uf") (at 227.33 69.85 90) (unit 1)
     (in_bom yes) (on_board yes)
-    (property "Reference" "C9" (id 0) (at 228.6 77.47 90))
-    (property "Value" "C_0805_10uf" (id 1) (at 228.6 74.93 90))
+    (property "Reference" "C9" (id 0) (at 214.63 72.39 90))
+    (property "Value" "C_0805_10uf" (id 1) (at 214.63 69.85 90))
     (property "Footprint" "footprints:C_0805_2012Metric" (id 2) (at 231.14 68.8848 0)
       (effects (font (size 1.27 1.27)) hide)
@@
     (pin "9")
   )
+  (symbol (lib_id "HPS:TestPoint") (at 237.49 87.63 180) (unit 1)
+    (in_bom yes) (on_board yes)
+    (property "Reference" "TP19" (id 0) (at 240.03 96.52 0)
+      (effects (font (size 1.27 1.27)) (justify left))
+    )
+    (property "Value" "TestPoint" (id 1) (at 240.03 93.98 0)
+      (effects (font (size 1.27 1.27)) (justify left))
+    )
+    (property "Footprint" "footprints:TestPoint_THTPad_D2.0mm_Drill1.0mm" (id 2) (at 232.41 87.63 0)
+      (effects (font (size 1.27 1.27)) hide)
+    )
+    (property "Datasheet" "~" (id 3) (at 232.41 87.63 0)
+      (effects (font (size 1.27 1.27)) hide)
+    )
+    (pin "1")
+  )
   (symbol (lib_id "HPS:GND") (at 72.39 273.05 0) (unit 1)
     (in_bom yes) (on_board yes) (fields_autoplaced)
@@
     (pin "2")
   )
+  (symbol (lib_id "HPS:TestPoint") (at 237.49 82.55 0) (unit 1)
+    (in_bom yes) (on_board yes)
+    (property "Reference" "TP18" (id 0) (at 232.41 73.66 0)
+      (effects (font (size 1.27 1.27)) (justify left))
+    )
+    (property "Value" "TestPoint" (id 1) (at 232.41 76.2 0)
+      (effects (font (size 1.27 1.27)) (justify left))
+    )
+    (property "Footprint" "footprints:TestPoint_THTPad_D2.0mm_Drill1.0mm" (id 2) (at 242.57 82.55 0)
+      (effects (font (size 1.27 1.27)) hide)
+    )
+    (property "Datasheet" "~" (id 3) (at 242.57 82.55 0)
+      (effects (font (size 1.27 1.27)) hide)
+    )
+    (pin "1")
+  )
   (symbol (lib_id "HPS:Omron_B3F_SPST") (at 182.88 193.04 90) (unit 1)
     (in_bom yes) (on_board yes) (fields_autoplaced)
@@
       (reference "TP16") (unit 1) (value "TestPoint") (footprint "footprints:TestPoint_THTPad_D2.0mm_Drill1.0mm")
     )
+    (path "/6110801d-482d-4ac3-b65e-9c89a9b29159"
+      (reference "TP17") (unit 1) (value "TestPoint") (footprint "footprints:TestPoint_THTPad_D2.0mm_Drill1.0mm")
+    )
+    (path "/d423b681-460c-43b7-8356-2af1eea02fad"
+      (reference "TP18") (unit 1) (value "TestPoint") (footprint "footprints:TestPoint_THTPad_D2.0mm_Drill1.0mm")
+    )
+    (path "/a08dab12-c869-4349-b3a1-0aa5e85405b5"
+      (reference "TP19") (unit 1) (value "TestPoint") (footprint "footprints:TestPoint_THTPad_D2.0mm_Drill1.0mm")
+    )
     (path "/0ddf550a-fb5a-4319-a932-814d21c1d496"

Commit message: Updated Schematic
Parts:
- removed J2: Power_inlet_vertical, footprints:Wurth-694106402002, symbol HPS:Power_inlet_vertical
- added J2: PJ-102AH, footprints:PJ-102AH, symbol HPS:PJ-102AH
Connections:
- net GND: now also J2.2 (OUT)
- net at C6.1, U3.1 (IN): now also J2.1 (POLE)
Changed lines of the file:
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@@
     (pin "2")
+  )
+  (symbol (lib_id "HPS:PJ-102AH") (at 35.56 265.43 0) (unit 1)
+    (in_bom yes) (on_board yes)
+    (property "Reference" "J2" (id 0) (at 33.02 252.73 0)
+      (effects (font (size 1.524 1.524)))
+    )
+    (property "Value" "PJ-102AH" (id 1) (at 33.02 256.54 0)
+      (effects (font (size 1.524 1.524)))
+    )
+    (property "Footprint" "footprints:PJ-102AH" (id 2) (at 33.02 260.35 0)
+      (effects (font (size 1.524 1.524)))
+    )
+    (property "Datasheet" "https://www.cuidevices.com/product/resource/pj-102ah.pdf" (id 3) (at 37.084 277.368 0)
+      (effects (font (size 1.524 1.524)) hide)
+    )
+    (property "MFG" "CUI Devices" (id 4) (at 35.56 283.21 0)
+      (effects (font (size 1.27 1.27)) hide)
+    )
+    (property "MPN" "PJ-102AH" (id 5) (at 35.56 285.75 0)
+      (effects (font (size 1.27 1.27)) hide)
+    )
+    (property "Digikey PN" "CP-102AH-ND" (id 6) (at 37.084 290.957 0)
+      (effects (font (size 1.27 1.27)) hide)
+    )
+    (property "Mouser PN" "490-PJ-102AH" (id 7) (at 35.56 288.163 0)
+      (effects (font (size 1.27 1.27)) hide)
+    )
+    (pin "1")
+    (pin "2")
+    (pin "3")
   )
   (symbol (lib_id "HPS:R_0805_47") (at 81.28 161.29 90) (unit 1)
@@
     (pin "1")
   )
-  (symbol (lib_id "HPS:Power_inlet_vertical") (at 35.56 265.43 0) (unit 1)
-    (in_bom yes) (on_board yes)
-    (property "Reference" "J2" (id 0) (at 22.86 267.97 90)
-      (effects (font (size 1.524 1.524)))
-    )
-    (property "Value" "Power_inlet_vertical" (id 1) (at 25.4 267.97 90)
-      (effects (font (size 1.524 1.524)))
-    )
-    (property "Footprint" "footprints:Wurth-694106402002" (id 2) (at 27.94 261.62 90)
-      (effects (font (size 1.524 1.524)))
-    )
-    (property "Datasheet" "https://www.we-online.com/katalog/datasheet/6941xx402002.pdf" (id 3) (at 37.084 277.368 0)
-      (effects (font (size 1.524 1.524)) hide)
-    )
-    (property "MFG" "Wurth" (id 4) (at 35.56 283.21 0)
-      (effects (font (size 1.27 1.27)) hide)
-    )
-    (property "MPN" "694106402002" (id 5) (at 35.56 285.75 0)
-      (effects (font (size 1.27 1.27)) hide)
-    )
-    (property "Digikey PN" "732-5931-ND" (id 6) (at 37.084 290.957 0)
-      (effects (font (size 1.27 1.27)) hide)
-    )
-    (pin "1")
-    (pin "2")
-    (pin "3")
-  )
   (symbol (lib_id "HPS:Buzzer") (at 68.58 207.01 0) (unit 1)
     (in_bom yes) (on_board yes)
@@
       (reference "J1") (unit 1) (value "Conn_01x06") (footprint "footprints:PinHeader_1x06_P2.54mm_Vertical")
     )
-    (path "/f2393e9d-3944-42e3-a465-3a363f1f67da"
-      (reference "J2") (unit 1) (value "Power_inlet_vertical") (footprint "footprints:Wurth-694106402002")
+    (path "/a64c7915-fcbf-4133-a2a7-a3d514957432"
+      (reference "J2") (unit 1) (value "PJ-102AH") (footprint "footprints:PJ-102AH")
     )
     (path "/62bfb222-688a-4806-adfa-d3b9a4604387"

Commit message: PCB and Schematic Fixes
Parts:
- removed TP17, TP18, TP19: TestPoint, footprints:TestPoint_THTPad_D2.0mm_Drill1.0mm, symbol HPS:TestPoint
Changed lines of the file:
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@@
   (junction (at 290.83 64.77) (diameter 0) (color 0 0 0 0)
   )
-  (junction (at 237.49 82.55) (diameter 0) (color 0 0 0 0)
-  )
   (junction (at 266.7 191.77) (diameter 0) (color 0 0 0 0)
   )
@@
   (junction (at 152.4 248.92) (diameter 0) (color 0 0 0 0)
   )
-  (junction (at 212.09 85.09) (diameter 0) (color 0 0 0 0)
-  )
   (junction (at 356.87 29.21) (diameter 0) (color 0 0 0 0)
   )
@@
   (junction (at 387.35 77.47) (diameter 0) (color 0 0 0 0)
   )
-  (junction (at 237.49 87.63) (diameter 0) (color 0 0 0 0)
-  )
   (junction (at 87.63 171.45) (diameter 0) (color 0 0 0 0)
   )
@@
     (stroke (width 0) (type default) (color 0 0 0 0))
   )
-  (wire (pts (xy 237.49 87.63) (xy 240.03 87.63))
-    (stroke (width 0) (type default) (color 0 0 0 0))
-  )
   (polyline (pts (xy 350.52 198.12) (xy 350.52 203.2))
     (stroke (width 0) (type default) (color 0 0 0 0))
@@
     (stroke (width 0) (type default) (color 0 0 0 0))
   )
-  (wire (pts (xy 237.49 82.55) (xy 240.03 82.55))
-    (stroke (width 0) (type default) (color 0 0 0 0))
-  )
   (wire (pts (xy 273.05 67.31) (xy 260.35 67.31))
     (stroke (width 0) (type default) (color 0 0 0 0))
@@
     (stroke (width 0) (type default) (color 0 0 0 0))
   )
-  (wire (pts (xy 209.55 85.09) (xy 212.09 85.09))
+  (wire (pts (xy 222.25 85.09) (xy 240.03 85.09))
     (stroke (width 0) (type default) (color 0 0 0 0))
   )
@@
     (stroke (width 0) (type default) (color 0 0 0 0))
   )
-  (wire (pts (xy 234.95 82.55) (xy 237.49 82.55))
+  (wire (pts (xy 234.95 82.55) (xy 240.03 82.55))
     (stroke (width 0) (type default) (color 0 0 0 0))
   )
@@
     (stroke (width 0) (type default) (color 0 0 0 0))
   )
-  (wire (pts (xy 233.68 87.63) (xy 237.49 87.63))
+  (wire (pts (xy 233.68 87.63) (xy 240.03 87.63))
     (stroke (width 0) (type default) (color 0 0 0 0))
   )
@@
     (stroke (width 0) (type default) (color 0 0 0 0))
   )
-  (wire (pts (xy 212.09 85.09) (xy 240.03 85.09))
-    (stroke (width 0) (type default) (color 0 0 0 0))
-  )
   (wire (pts (xy 356.87 64.77) (xy 356.87 29.21))
     (stroke (width 0) (type default) (color 0 0 0 0))
@@
     )
   )
-  (global_label "LED_SCK" (shape input) (at 209.55 85.09 180) (fields_autoplaced)
+  (global_label "LED_SCK" (shape input) (at 222.25 85.09 180) (fields_autoplaced)
     (effects (font (size 1.27 1.27)) (justify right))
-    (property "Intersheet References" "${INTERSHEET_REFS}" (id 0) (at 198.9726 85.0106 0)
+    (property "Intersheet References" "${INTERSHEET_REFS}" (id 0) (at 211.6726 85.0106 0)
       (effects (font (size 1.27 1.27)) (justify right) hide)
     )
@@
     (pin "2")
   )
+  (symbol (lib_id "HPS:PJ-102AH") (at 35.56 265.43 0) (unit 1)
+    (in_bom yes) (on_board yes) (fields_autoplaced)
+    (property "Reference" "J2" (id 0) (at 33.02 252.73 0)
+      (effects (font (size 1.524 1.524)))
+    )
+    (property "Value" "PJ-102AH" (id 1) (at 33.02 256.54 0)
+      (effects (font (size 1.524 1.524)))
+    )
+    (property "Footprint" "footprints:PJ-102AH" (id 2) (at 33.02 260.35 0)
+      (effects (font (size 1.524 1.524)))
+    )
+    (property "Datasheet" "https://www.cuidevices.com/product/resource/pj-102ah.pdf" (id 3) (at 37.084 277.368 0)
+      (effects (font (size 1.524 1.524)) hide)
+    )
+    (property "MFG" "CUI Devices" (id 4) (at 35.56 283.21 0)
+      (effects (font (size 1.27 1.27)) hide)
+    )
+    (property "MPN" "PJ-102AH" (id 5) (at 35.56 285.75 0)
+      (effects (font (size 1.27 1.27)) hide)
+    )
+    (property "Digikey PN" "CP-102AH-ND" (id 6) (at 37.084 290.957 0)
+      (effects (font (size 1.27 1.27)) hide)
+    )
+    (property "Mouser PN" "490-PJ-102AH" (id 7) (at 35.56 288.163 0)
+      (effects (font (size 1.27 1.27)) hide)
+    )
+    (pin "1")
+    (pin "2")
+    (pin "3")
+  )
   (symbol (lib_id "HPS:GND") (at 256.54 130.81 0) (unit 1)
     (in_bom yes) (on_board yes) (fields_autoplaced)
@@
     (pin "1")
   )
-  (symbol (lib_id "HPS:TestPoint") (at 212.09 85.09 0) (unit 1)
-    (in_bom yes) (on_board yes)
-    (property "Reference" "TP17" (id 0) (at 209.55 76.2 0)
-      (effects (font (size 1.27 1.27)) (justify left))
-    )
-    (property "Value" "TestPoint" (id 1) (at 209.55 78.74 0)
-      (effects (font (size 1.27 1.27)) (justify left))
-    )
-    (property "Footprint" "footprints:TestPoint_THTPad_D2.0mm_Drill1.0mm" (id 2) (at 217.17 85.09 0)
-      (effects (font (size 1.27 1.27)) hide)
-    )
-    (property "Datasheet" "~" (id 3) (at 217.17 85.09 0)
-      (effects (font (size 1.27 1.27)) hide)
-    )
-    (pin "1")
-  )
   (symbol (lib_id "HPS:Crystal_32768Hz") (at 276.86 198.12 270) (unit 1)
     (in_bom yes) (on_board yes)
@@
   (symbol (lib_id "HPS:C_0805_10uf") (at 227.33 69.85 90) (unit 1)
     (in_bom yes) (on_board yes)
-    (property "Reference" "C9" (id 0) (at 214.63 72.39 90))
-    (property "Value" "C_0805_10uf" (id 1) (at 214.63 69.85 90))
+    (property "Reference" "C9" (id 0) (at 228.6 77.47 90))
+    (property "Value" "C_0805_10uf" (id 1) (at 228.6 74.93 90))
     (property "Footprint" "footprints:C_0805_2012Metric" (id 2) (at 231.14 68.8848 0)
       (effects (font (size 1.27 1.27)) hide)
@@
     (pin "9")
   )
-  (symbol (lib_id "HPS:TestPoint") (at 237.49 87.63 180) (unit 1)
-    (in_bom yes) (on_board yes)
-    (property "Reference" "TP19" (id 0) (at 240.03 96.52 0)
-      (effects (font (size 1.27 1.27)) (justify left))
-    )
-    (property "Value" "TestPoint" (id 1) (at 240.03 93.98 0)
-      (effects (font (size 1.27 1.27)) (justify left))
-    )
-    (property "Footprint" "footprints:TestPoint_THTPad_D2.0mm_Drill1.0mm" (id 2) (at 232.41 87.63 0)
-      (effects (font (size 1.27 1.27)) hide)
-    )
-    (property "Datasheet" "~" (id 3) (at 232.41 87.63 0)
-      (effects (font (size 1.27 1.27)) hide)
-    )
-    (pin "1")
-  )
   (symbol (lib_id "HPS:GND") (at 72.39 273.05 0) (unit 1)
     (in_bom yes) (on_board yes) (fields_autoplaced)
@@
     (pin "2")
   )
-  (symbol (lib_id "HPS:PJ-102AH") (at 35.56 265.43 0) (unit 1)
-    (in_bom yes) (on_board yes)
-    (property "Reference" "J2" (id 0) (at 33.02 252.73 0)
-      (effects (font (size 1.524 1.524)))
-    )
-    (property "Value" "PJ-102AH" (id 1) (at 33.02 256.54 0)
-      (effects (font (size 1.524 1.524)))
-    )
-    (property "Footprint" "footprints:PJ-102AH" (id 2) (at 33.02 260.35 0)
-      (effects (font (size 1.524 1.524)))
-    )
-    (property "Datasheet" "https://www.cuidevices.com/product/resource/pj-102ah.pdf" (id 3) (at 37.084 277.368 0)
-      (effects (font (size 1.524 1.524)) hide)
-    )
-    (property "MFG" "CUI Devices" (id 4) (at 35.56 283.21 0)
-      (effects (font (size 1.27 1.27)) hide)
-    )
-    (property "MPN" "PJ-102AH" (id 5) (at 35.56 285.75 0)
-      (effects (font (size 1.27 1.27)) hide)
-    )
-    (property "Digikey PN" "CP-102AH-ND" (id 6) (at 37.084 290.957 0)
-      (effects (font (size 1.27 1.27)) hide)
-    )
-    (property "Mouser PN" "490-PJ-102AH" (id 7) (at 35.56 288.163 0)
-      (effects (font (size 1.27 1.27)) hide)
-    )
-    (pin "1")
-    (pin "2")
-    (pin "3")
-  )
   (symbol (lib_id "HPS:R_0805_47") (at 81.28 161.29 90) (unit 1)
     (in_bom yes) (on_board yes) (fields_autoplaced)
@@
     (pin "2")
   )
-  (symbol (lib_id "HPS:TestPoint") (at 237.49 82.55 0) (unit 1)
-    (in_bom yes) (on_board yes)
-    (property "Reference" "TP18" (id 0) (at 232.41 73.66 0)
-      (effects (font (size 1.27 1.27)) (justify left))
-    )
-    (property "Value" "TestPoint" (id 1) (at 232.41 76.2 0)
-      (effects (font (size 1.27 1.27)) (justify left))
-    )
-    (property "Footprint" "footprints:TestPoint_THTPad_D2.0mm_Drill1.0mm" (id 2) (at 242.57 82.55 0)
-      (effects (font (size 1.27 1.27)) hide)
-    )
-    (property "Datasheet" "~" (id 3) (at 242.57 82.55 0)
-      (effects (font (size 1.27 1.27)) hide)
-    )
-    (pin "1")
-  )
   (symbol (lib_id "HPS:Omron_B3F_SPST") (at 182.88 193.04 90) (unit 1)
     (in_bom yes) (on_board yes) (fields_autoplaced)
@@
       (reference "J1") (unit 1) (value "Conn_01x06") (footprint "footprints:PinHeader_1x06_P2.54mm_Vertical")
     )
-    (path "/a64c7915-fcbf-4133-a2a7-a3d514957432"
+    (path "/1cdda1e7-f2a6-4dbd-86ac-4841a6c8e98a"
       (reference "J2") (unit 1) (value "PJ-102AH") (footprint "footprints:PJ-102AH")
     )
@@
       (reference "TP16") (unit 1) (value "TestPoint") (footprint "footprints:TestPoint_THTPad_D2.0mm_Drill1.0mm")
     )
-    (path "/6110801d-482d-4ac3-b65e-9c89a9b29159"
-      (reference "TP17") (unit 1) (value "TestPoint") (footprint "footprints:TestPoint_THTPad_D2.0mm_Drill1.0mm")
-    )
-    (path "/d423b681-460c-43b7-8356-2af1eea02fad"
-      (reference "TP18") (unit 1) (value "TestPoint") (footprint "footprints:TestPoint_THTPad_D2.0mm_Drill1.0mm")
-    )
-    (path "/a08dab12-c869-4349-b3a1-0aa5e85405b5"
-      (reference "TP19") (unit 1) (value "TestPoint") (footprint "footprints:TestPoint_THTPad_D2.0mm_Drill1.0mm")
-    )
     (path "/0ddf550a-fb5a-4319-a932-814d21c1d496"
