File: Annahs_clock_hps/Annahs_clock_hps.kicad_pcb (KiCad board)
At the start: 2 copper layers, 140 x 90 mm, 4 parts

Commit message: Updated Schematic and PCB
Parts:
- added BT1: Battery_Cell, footprints:BatteryHolder_Keystone_106_1x20mm, F.Cu at (90.0, 73.7)
- added BZ1: Buzzer, footprints:Buzzer_TDK_PS1240P02BT_D12.2mm_H6.5mm, F.Cu at (193.0, 66.0)
- added C1: C_0805_0.1uf, footprints:C_0805_2012Metric, F.Cu at (208.3, 132.1)
- added C2: C_0805_0.1uf, footprints:C_0805_2012Metric, F.Cu at (198.1, 106.7)
- added C3: C_0805_0.1uf, footprints:C_0805_2012Metric, F.Cu at (132.1, 88.9)
- added C4: C_0805_22pf, footprints:C_0805_2012Metric, F.Cu at (142.2, 137.2)
- added C5: C_0805_22pf, footprints:C_0805_2012Metric, F.Cu at (198.1, 96.5)
- added C6: C_0805_1uf, footprints:C_0805_2012Metric, F.Cu at (200.7, 129.5)
- added C7: C_0805_0.1uf, footprints:C_0805_2012Metric, F.Cu at (185.4, 71.1)
- added C8: C_0805_0.1uf, footprints:C_0805_2012Metric, F.Cu at (185.4, 81.3)
- added C9: C_0805_10uf, footprints:C_0805_2012Metric, F.Cu at (88.9, 129.5)
- added D1: LED_0805, footprints:LED_0805_2012Metric, F.Cu at (162.6, 88.9)
- added DS1: TC1602A-01T, footprints:TC1602A-01T, F.Cu at (117.9, 96.4)
- added J1: Conn_01x06, footprints:PinHeader_1x06_P2.54mm_Vertical, F.Cu at (104.1, 92.7)
- added J2: Power_inlet_vertical, footprints:Wurth-694106402002, F.Cu at (101.6, 132.1)
- added R1: R_0805_10K, footprints:R_0805_2012Metric, F.Cu at (199.0, 114.3)
- added R10: R_0805_100K, footprints:R_0805_2012Metric, F.Cu at (121.9, 88.9)
- added R11: R_0805_2.2K, footprints:R_0805_2012Metric, F.Cu at (149.9, 88.9)
- added R2: R_0805_10K, footprints:R_0805_2012Metric, F.Cu at (199.8, 121.9)
- added R3: R_0805_4.7K, footprints:R_0805_2012Metric, F.Cu at (177.8, 86.4)
- added R4: R_0805_4.7K, footprints:R_0805_2012Metric, F.Cu at (142.2, 88.9)
- added R5: R_0805_10K, footprints:R_0805_2012Metric, F.Cu at (185.4, 63.5)
- added R6: R_0805_4.7K, footprints:R_0805_2012Metric, F.Cu at (198.1, 91.4)
- added R7: R_0805_4.7K, footprints:R_0805_2012Metric, F.Cu at (208.3, 66.0)
- added R8: R_0805_10K, footprints:R_0805_2012Metric, F.Cu at (208.3, 111.8)
- added R9: R_0805_10K, footprints:R_0805_2012Metric, F.Cu at (213.4, 127.0)
- added RV1: R_POT_10K, footprints:Potentiometer_Bourns_3386P_Vertical, F.Cu at (208.3, 121.9)
- added SW1: Omron_B3F_SPST, footprints:SW_SPST_Omron_B3FS-100xP, F.Cu at (149.9, 137.2)
- added SW2: Omron_B3F_SPST, footprints:SW_SPST_Omron_B3FS-100xP, F.Cu at (162.6, 137.2)
- added SW3: Omron_B3F_SPST, footprints:SW_SPST_Omron_B3FS-100xP, F.Cu at (175.3, 137.2)
- added SW4: Omron_B3F_SPST, footprints:SW_SPST_Omron_B3FS-100xP, F.Cu at (188.0, 137.2)
- added SW5: Omron_B3F_SPST, footprints:SW_SPST_Omron_B3FS-100xP, F.Cu at (200.7, 137.2)
- added U1: DS1307_DIP-8, footprints:DIP-8_W7.62mm, F.Cu at (189.2, 77.4)
- added U2: MAX7219, footprints:DIP-24_W7.62mm, F.Cu at (87.6, 95.2)
- added U3: L7805, footprints:TO-220-3_Vertical, F.Cu at (114.3, 137.2)
- added U4: SC56-11EWA, footprints:Sx56-1xxxxx, F.Cu at (165.2, 78.6)
- added U5: SC56-11EWA, footprints:Sx56-1xxxxx, F.Cu at (127.1, 78.6)
- added UI1: ATmega328-PU, footprints:DIP-28_W7.62mm, F.Cu at (204.5, 72.4)
- added Y1: Crystal_16MHz, footprints:Crystal_SMD_HC49-SD, F.Cu at (131.2, 137.2)
- added Y2: Crystal_32768Hz, footprints:Crystal_SMD_2Pin_3.2x1.5mm, F.Cu at (185.4, 88.9)
