File: Annahs_clock_hps/Annahs_clock_hps.kicad_pcb (KiCad board)
At the start: 2 copper layers, 140 x 90 mm, 71 parts, among them J1 Conn_01x06, J2 Power_inlet_vertical, J3 Conn_02x03_Odd_Even, Q1 NPN_2N3904_SOT23, SW1 Omron_B3F_SPST, SW2 Omron_B3F_SPST, SW3 Omron_B3F_SPST, SW4 Omron_B3F_SPST, SW5 Omron_B3F_SPST, SW6 Omron_B3F_SPST, U1 DS1307_DIP-8, U2 MAX7219, U3 L7805, U4 SC56-11EWA, U5 SC56-11EWA, Y1 Crystal_16MHz, Y2 Crystal_32768Hz

Commit message: Undo Re-Organization
Parts:
- moved C6 1.72 mm to (203.6, 127.0)
- moved C7 1.72 mm to (203.0, 140.3)
- moved U3 1.72 mm to (204.9, 134.0)
- moved J2 1.72 mm to (190.2, 137.4)
Other:
- rule pad_to_mask_clearance: 0 -> 0.0762

Commit message: Updated Schematic and PCB
Parts:
- added R18: R_0805_1K, footprints:R_0805_2012Metric, F.Cu at (191.8, 71.1)
- R14: value R_0805_2.2K -> R_0805_1K
- moved C6 1.20 mm to (202.4, 127.0)
- moved C7 1.20 mm to (201.8, 140.3)
- moved U3 1.20 mm to (203.7, 134.0)
Connections:
- net /Buzzer renamed Buzzer
- net /Down_SW renamed Down_SW
- net /Driver_Load renamed MAX_Load
- net /LCD_Data4 renamed LCD_D4
- net /LCD_Data5 renamed LCD_D5
- net /LCD_Data6 renamed LCD_D6
- net /LCD_Data7 renamed LCD_D7
- net /LCD_Enable renamed LCD_E
- net /LCD_RS renamed LCD_RS
- net /RTC_SCL renamed RTC_SCL
- net /RTC_SDA renamed RTC_SDA
- net /Select_SW renamed Select_SW
- net /Up_SW renamed Up_SW
- net MISO renamed Alarm_SW
- net MOSI renamed MAX_DIN
- BZ1 pad 2: GND -> Net-(BZ1-Pad2)
- Q1 pad 3: GND -> Net-(BZ1-Pad2)
- TP13 pad 1: GND -> Net-(BZ1-Pad2)
Routing:
- net Net-(BZ1-Pad2): track 0.00 -> 33.6 mm, vias 0 -> 2
- net GND: track 210.3 -> 184.7 mm, vias 20 -> 18
- net Buzzer: track 27.9 -> 30.1 mm
- net Down_SW: track 136.5 -> 135.0 mm
- net /Dig01_C: track 98.7 -> 97.3 mm
- net Net-(C6-Pad1): track 18.1 -> 16.9 mm
- net /Dig01_A: track 100.8 -> 101.8 mm
- net TXD: track 45.9 -> 45.0 mm

Commit message: Updated PCB and Schematic
Parts:
- added TP15: TestPoint, footprints:TestPoint_THTPad_D2.0mm_Drill1.0mm, F.Cu at (86.1, 90.7)
- added TP16: TestPoint, footprints:TestPoint_THTPad_D2.0mm_Drill1.0mm, F.Cu at (86.6, 96.3)
Routing:
- net RTC_SDA: track 146.1 -> 173.8 mm, vias 2 -> 3
- net RTC_SCL: track 147.5 -> 174.7 mm, vias 2 -> 3
Changed lines of the file:
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@@
       (net 54 "/Dig01_C") (pinfunction "1") (pintype "passive"))
   )
+  (footprint "footprints:TestPoint_THTPad_D2.0mm_Drill1.0mm" (layer "F.Cu")
+    (at 86.614 96.266)
+    (descr "THT pad as test Point, diameter 2.0mm, hole diameter 1.0mm")
+    (tags "test point THT pad")
+    (property "Sheetfile" "Annahs_clock_hps.kicad_sch")
+    (property "Sheetname" "")
+    (attr exclude_from_pos_files)
+    (fp_text reference "TP16" (at 0 -1.998) (layer "F.SilkS")
+      (effects (font (size 1 1) (thickness 0.15)))
+    )
+    (fp_text value "TestPoint" (at 0 2.05) (layer "F.Fab")
+      (effects (font (size 1 1) (thickness 0.15)))
+    )
+    (fp_text user "${REFERENCE}" (at 0 -2) (layer "F.Fab")
+      (effects (font (size 1 1) (thickness 0.15)))
+    )
+    (fp_circle (center 0 0) (end 0 1.2) (layer "F.SilkS") (width 0.12) (fill none))
+    (fp_circle (center 0 0) (end 1.5 0) (layer "F.CrtYd") (width 0.05) (fill none))
+    (pad "1" thru_hole circle (at 0 0) (size 2 2) (drill 1) (layers *.Cu *.Mask)
+      (net 37 "RTC_SDA") (pinfunction "1") (pintype "passive"))
+  )
   (footprint "footprints:R_0805_2012Metric" (layer "F.Cu")
     (at 164.465 140.0175 -90)
@@
     )
   )
+  (footprint "footprints:TestPoint_THTPad_D2.0mm_Drill1.0mm" (layer "F.Cu")
+    (at 86.106 90.678)
+    (descr "THT pad as test Point, diameter 2.0mm, hole diameter 1.0mm")
+    (tags "test point THT pad")
+    (property "Sheetfile" "Annahs_clock_hps.kicad_sch")
+    (property "Sheetname" "")
+    (attr exclude_from_pos_files)
+    (fp_text reference "TP15" (at 0 -1.998) (layer "F.SilkS")
+      (effects (font (size 1 1) (thickness 0.15)))
+    )
+    (fp_text value "TestPoint" (at 0 2.05) (layer "F.Fab")
+      (effects (font (size 1 1) (thickness 0.15)))
+    )
+    (fp_text user "${REFERENCE}" (at 0 -2) (layer "F.Fab")
+      (effects (font (size 1 1) (thickness 0.15)))
+    )
+    (fp_circle (center 0 0) (end 0 1.2) (layer "F.SilkS") (width 0.12) (fill none))
+    (fp_circle (center 0 0) (end 1.5 0) (layer "F.CrtYd") (width 0.05) (fill none))
+    (pad "1" thru_hole circle (at 0 0) (size 2 2) (drill 1) (layers *.Cu *.Mask)
+      (net 60 "RTC_SCL") (pinfunction "1") (pintype "passive"))
+  )
   (footprint "footprints:C_0805_2012Metric" (layer "F.Cu")
     (at 165.315 135.1525 180)
@@
     (property "Sheetname" "")
     (attr smd)
-    (fp_text reference "U1" (at 3.81 -2.33 90) (layer "F.SilkS")
+    (fp_text reference "U1" (at 6.604 -2.296 90) (layer "F.SilkS")
       (effects (font (size 1 1) (thickness 0.15)))
     )
@@
   (segment (start 177.355 140.68) (end 169.355 140.68) (width 0.2032) (layer "F.Cu") (net 36))
   (segment (start 180.975 140.55) (end 177.485 140.55) (width 0.2032) (layer "F.Cu") (net 36))
+  (segment (start 86.614 96.266) (end 88.9 93.98) (width 0.2032) (layer "F.Cu") (net 37))
   (segment (start 93.345 71.12) (end 92.72 71.12) (width 0.2032) (layer "F.Cu") (net 37))
   (segment (start 94.83 60.11) (end 95.885 59.055) (width 0.2032) (layer "F.Cu") (net 37))
@@
   (segment (start 210.82 74.295) (end 208.28 76.835) (width 0.2032) (layer "F.Cu") (net 37))
   (segment (start 94.83 67.31) (end 94.83 60.11) (width 0.2032) (layer "F.Cu") (net 37))
+  (segment (start 88.9 77.724) (end 90.932 75.692) (width 0.2032) (layer "F.Cu") (net 37))
+  (segment (start 88.9 93.98) (end 88.9 77.724) (width 0.2032) (layer "F.Cu") (net 37))
   (segment (start 93.345 71.12) (end 94.615 69.85) (width 0.2032) (layer "F.Cu") (net 37))
   (segment (start 94.615 69.85) (end 94.615 67.525) (width 0.2032) (layer "F.Cu") (net 37))
   (via (at 95.885 59.055) (size 0.8128) (drill 0.4064) (layers "F.Cu" "B.Cu") (net 37))
+  (via (at 90.932 75.692) (size 0.8) (drill 0.4) (layers "F.Cu" "B.Cu") (net 37))
   (via (at 210.82 63.5) (size 0.8128) (drill 0.4064) (layers "F.Cu" "B.Cu") (net 37))
+  (segment (start 92.72 71.12) (end 92.72 73.904) (width 0.2032) (layer "B.Cu") (net 37))
   (segment (start 205.96909 58.64909) (end 210.82 63.5) (width 0.2032) (layer "B.Cu") (net 37))
+  (segment (start 92.72 73.904) (end 90.932 75.692) (width 0.2032) (layer "B.Cu") (net 37))
   (segment (start 96.29091 58.64909) (end 205.96909 58.64909) (width 0.2032) (layer "B.Cu") (net 37))
   (segment (start 95.885 59.055) (end 96.29091 58.64909) (width 0.2032) (layer "B.Cu") (net 37))
@@
   (segment (start 144.855701 85.165701) (end 145.415 85.725) (width 0.2032) (layer "B.Cu") (net 59))
   (segment (start 130.885701 85.165701) (end 130.81 85.09) (width 0.2032) (layer "B.Cu") (net 59))
+  (segment (start 83.058 87.63) (end 86.106 90.678) (width 0.2032) (layer "F.Cu") (net 60))
   (segment (start 90.18 71.12) (end 90.18 69.84) (width 0.2032) (layer "F.Cu") (net 60))
   (segment (start 90.18 69.84) (end 90.805 69.215) (width 0.2032) (layer "F.Cu") (net 60))
   (segment (start 90.805 69.215) (end 90.805 67.31) (width 0.2032) (layer "F.Cu") (net 60))
   (segment (start 209.55 59.69) (end 209.55 72.39) (width 0.2032) (layer "F.Cu") (net 60))
+  (segment (start 83.058 75.184) (end 83.058 87.63) (width 0.2032) (layer "F.Cu") (net 60))
   (segment (start 90.805 67.31) (end 90.805 59.055) (width 0.2032) (layer "F.Cu") (net 60))
   (segment (start 208.27 73.67) (end 207.655 73.67) (width 0.2032) (layer "F.Cu") (net 60))
@@
   (via (at 209.55 59.69) (size 0.8128) (drill 0.4064) (layers "F.Cu" "B.Cu") (net 60))
   (via (at 92.075 57.785) (size 0.8128) (drill 0.4064) (layers "F.Cu" "B.Cu") (net 60))
+  (via (at 83.058 75.184) (size 0.8) (drill 0.4) (layers "F.Cu" "B.Cu") (net 60))
+  (segment (start 90.18 73.904) (end 88.9 75.184) (width 0.2032) (layer "B.Cu") (net 60))
+  (segment (start 88.9 75.184) (end 83.058 75.184) (width 0.2032) (layer "B.Cu") (net 60))
   (segment (start 92.075 57.785) (end 207.645 57.785) (width 0.2032) (layer "B.Cu") (net 60))
   (segment (start 207.645 57.785) (end 209.55 59.69) (width 0.2032) (layer "B.Cu") (net 60))
+  (segment (start 90.18 71.12) (end 90.18 73.904) (width 0.2032) (layer "B.Cu") (net 60))
   (segment (start 187.96 80.645) (end 191.77 80.645) (width 0.2032) (layer "F.Cu") (net 64))
   (segment (start 186.055 63.715) (end 186.055 73.66) (width 0.2032) (layer "F.Cu") (net 64))

Commit message: Schematic and PCB Update
Parts:
- added TP17: TestPoint, footprints:TestPoint_THTPad_D2.0mm_Drill1.0mm, F.Cu at (103.9, 120.7)
- added TP18: TestPoint, footprints:TestPoint_THTPad_D2.0mm_Drill1.0mm, F.Cu at (104.1, 110.0)
- added TP19: TestPoint, footprints:TestPoint_THTPad_D2.0mm_Drill1.0mm, F.Cu at (104.1, 115.3)
- moved TP12 0.99 mm to (214.6, 132.6)
- moved TP2 0.97 mm to (214.4, 128.5)
Connections:
- net Alarm_SW renamed MISO
- net MAX_DIN renamed MOSI
Routing:
- net LED_SCK: track 177.7 -> 217.9 mm, vias 4 -> 6
- net MAX_Load: track 143.3 -> 160.4 mm
- net MOSI: track 140.1 -> 154.4 mm

Commit message: Updated Schematic and PCB
Parts:
- moved TP11 6.10 mm to (120.0, 79.8)
Routing:
- net /Dig01_F: track 83.2 -> 79.7 mm, vias 5 -> 4
- net /Dig01_G: track 101.4 -> 104.9 mm
- net /Dig0_Com: track 88.9 -> 85.4 mm
- net Buzzer: track 30.1 -> 27.0 mm
- net /Dig01_B: track 101.0 -> 104.0 mm
- net /Dig01_A: track 101.8 -> 99.2 mm
- net LCD_D6: track 62.0 -> 63.7 mm
- net /Dig01_C: track 97.3 -> 99.0 mm
- net LCD_E: track 85.5 -> 87.1 mm
- net MOSI: track 154.4 -> 152.8 mm
- net LCD_D7: track 70.8 -> 72.4 mm
- net /Dig01_DP: track 83.1 -> 84.7 mm
- net TXD: track 45.0 -> 46.3 mm
- net Down_SW: track 135.0 -> 136.1 mm
- net /Dig01_D: track 96.5 -> 97.5 mm
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
Commit message: Updated PCB/Schematic/Gerber
Parts:
- J2: value Power_inlet_vertical -> PJ-102AH; footprint footprints:Wurth-694106402002 -> footprints:PJ-102AH
- moved R9 4.05 mm to (158.2, 137.0), turned to 90 degrees
- moved J2 3.21 mm to (193.2, 136.1)
- moved C11 2.04 mm to (165.2, 133.1)
- moved R13 2.04 mm to (164.3, 138.0)
- moved SW1 2.04 mm to (173.2, 136.4)
- moved R2 2.04 mm to (180.8, 137.7)
- moved R15 2.03 mm to (142.0, 138.9)
- moved SW4 2.03 mm to (149.9, 136.4)
- moved C13 2.03 mm to (142.2, 133.9)
- moved R12 1.40 mm to (118.5, 138.9)
- moved R1 1.40 mm to (134.3, 138.3)
- moved SW2 1.40 mm to (126.5, 136.4)
- moved C10 1.40 mm to (118.7, 133.9)
- moved R8 1.40 mm to (110.5, 138.1)
- moved SW3 1.40 mm to (102.9, 136.4)
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Routing:
- net Net-(C6-Pad1): track 16.9 -> 13.5 mm
- net Net-(R15-Pad2): track 13.8 -> 15.8 mm
- net RXD: track 49.5 -> 47.8 mm
- net /Dig0_Com: track 85.4 -> 83.9 mm
- net MOSI: track 152.8 -> 151.4 mm
- net MISO: track 169.8 -> 168.4 mm
- net /Dig1_Com: track 173.5 -> 172.1 mm
- net Down_SW: track 136.1 -> 134.8 mm
- net Select_SW: track 73.0 -> 72.0 mm
- net /Dig01_A: track 99.2 -> 100.1 mm
