File: Annahs_clock_hps/Annahs_clock_hps.kicad_pcb (KiCad board)
At the start: 2 copper layers, 140 x 90 mm, 77 parts, among them J1 Conn_01x06, J2 PJ-102AH, J3 Conn_02x03_Odd_Even, Q1 NPN_2N3904_SOT23, SW1 Omron_B3F_SPST, SW2 Omron_B3F_SPST, SW3 Omron_B3F_SPST, SW4 Omron_B3F_SPST, SW5 Omron_B3F_SPST, SW6 Omron_B3F_SPST, U1 DS1307_DIP-8, U2 MAX7219, U3 L7805, U4 SC56-11EWA, U5 SC56-11EWA, Y1 Crystal_16MHz, Y2 Crystal_32768Hz

Commit message: PCB and Schematic Fixes
Parts:
- removed TP17, TP18, TP19: TestPoint, footprints:TestPoint_THTPad_D2.0mm_Drill1.0mm
- moved TP11 6.10 mm to (120.0, 73.7)
- moved R9 4.05 mm to (157.5, 141.0), turned to 0 degrees
- moved C11 2.04 mm to (165.3, 135.2)
- moved R13 2.04 mm to (164.5, 140.0)
- moved SW1 2.04 mm to (173.4, 138.4)
- moved R2 2.04 mm to (181.0, 139.7)
- moved R15 2.03 mm to (142.0, 141.0)
- moved SW4 2.03 mm to (149.9, 138.4)
- moved C13 2.03 mm to (142.2, 135.9)
- moved R12 1.40 mm to (118.3, 140.3)
- moved R1 1.40 mm to (134.2, 139.7)
- moved SW2 1.40 mm to (126.4, 137.8)
- moved C10 1.40 mm to (118.5, 135.3)
- moved R8 1.40 mm to (110.5, 139.5)
- moved SW3 1.40 mm to (102.9, 137.8)
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Routing:
- net LED_SCK: track 217.9 -> 177.7 mm, vias 6 -> 4
- net MAX_Load: track 159.7 -> 143.3 mm
- net MOSI: track 151.4 -> 140.1 mm
- net /Dig0_Com: track 83.9 -> 88.7 mm
- net /Dig01_F: track 79.7 -> 83.2 mm, vias 4 -> 5
- net /Dig01_G: track 104.9 -> 101.4 mm
- net Buzzer: track 27.0 -> 30.1 mm
- net /Dig01_B: track 104.0 -> 101.0 mm
- net Net-(R15-Pad2): track 15.8 -> 13.8 mm
- net LCD_D6: track 63.7 -> 62.0 mm
- net RXD: track 47.8 -> 49.5 mm
- net /Dig01_C: track 99.0 -> 97.3 mm
- net /Dig01_A: track 100.1 -> 101.8 mm
- net LCD_E: track 87.1 -> 85.5 mm
- net LCD_D7: track 72.4 -> 70.8 mm
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
Commit message: PCB and Schematic Updates
Parts:
- J2: value PJ-102AH -> VAL**
- moved R9 1.18 mm to (157.5, 139.8), turned to 90 degrees
- moved C2 0.44 mm to (210.8, 91.0)
Routing:
- net Net-(R15-Pad2): track 13.8 -> 14.7 mm
