File: Annahs_clock_hps/_autosave-Annahs_clock_hps.kicad_pcb (KiCad board)
At the start: 2 copper layers, 140 x 90 mm, 77 parts, among them J1 Conn_01x06, J2 Power_inlet_vertical, J3 Conn_02x03_Odd_Even, Q1 NPN_2N3904_SOT23, SW1 Omron_B3F_SPST, SW2 Omron_B3F_SPST, SW3 Omron_B3F_SPST, SW4 Omron_B3F_SPST, SW5 Omron_B3F_SPST, SW6 Omron_B3F_SPST, U1 DS1307_DIP-8, U2 MAX7219, U3 L7805, U4 SC56-11EWA, U5 SC56-11EWA, Y1 Crystal_16MHz, Y2 Crystal_32768Hz

Commit message: Updated Schematic
Parts:
- J2: value Power_inlet_vertical -> PJ-102AH; footprint footprints:Wurth-694106402002 -> footprints:PJ-102AH
- moved R9 4.05 mm to (158.2, 137.0), turned to 90 degrees
- moved J2 3.22 mm to (193.1, 136.1)
- moved C11 2.04 mm to (165.2, 133.1)
- moved R13 2.04 mm to (164.3, 138.0)
- moved SW1 2.04 mm to (173.2, 136.4)
- moved R2 2.04 mm to (180.8, 137.7)
- moved R15 2.03 mm to (142.0, 138.9)
- moved SW4 2.03 mm to (149.9, 136.4)
- moved C13 2.03 mm to (142.2, 133.9)
- moved R12 1.40 mm to (118.5, 138.9)
- moved R1 1.40 mm to (134.3, 138.3)
- moved SW2 1.40 mm to (126.5, 136.4)
- moved C10 1.40 mm to (118.7, 133.9)
- moved R8 1.40 mm to (110.5, 138.1)
- moved SW3 1.40 mm to (102.9, 136.4)
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Routing:
- net Net-(C6-Pad1): track 16.9 -> 13.5 mm
- net Net-(R15-Pad2): track 13.8 -> 15.8 mm
- net RXD: track 49.5 -> 47.8 mm
- net /Dig0_Com: track 85.4 -> 83.9 mm
- net Select_SW: track 73.0 -> 71.5 mm
- net MOSI: track 152.8 -> 151.4 mm
- net /Dig1_Com: track 173.5 -> 172.1 mm
- net Down_SW: track 136.1 -> 134.8 mm
- net MISO: track 169.8 -> 168.7 mm
- net /Dig01_A: track 99.2 -> 100.1 mm
