File: Annahs_clock_hps/Annahs_clock_hps-backups/Annahs_clock_hps-2022-06-10_130227/Annahs_clock_hps.kicad_sch (KiCad schematic)
At the start: 10 parts, among them SW1 Omron_B3F_SPST, SW2 Omron_B3F_SPST, SW3 Omron_B3F_SPST, SW4 Omron_B3F_SPST, U1 DS1307_DIP-8, U2 MAX7219

Commit message: Clock Schematic
Parts:
- added DS2: LED_Display_1001, footprints:Adafruit-1001-0-0-MFG, symbol HPS:LED_Display_1001
Connections:
- net GND: now also U2.4 (GND), U2.9 (GND)
- net VCC: now also U2.19 (V+)
- net at U2.14 (SEG_A): now also DS2.13 (A)
- net at U2.15 (SEG_F): now also DS2.12 (F)
- net at U2.16 (SEG_B): now also DS2.9 (B)
- net at U2.17 (SEG_G): now also DS2.5 (G)
- net at U2.20 (SEG_C): now also DS2.4 (C)
- net at U2.21 (SEG_E): now also DS2.1 (E)
- net at U2.22 (SEG_DP): now also DS2.3 (DP)
- net at U2.23 (SEG_D): now also DS2.2 (D)
Other:
- moved on the sheet: U1

Commit message: Clock Schematic
Connections:
- net at DS2.14 (COM_DIG.1): now also U2.11 (DIG_1)
Changed lines of the file:
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@@
+    (stroke (width 0) (type default) (color 0 0 0 0))
+  )
+  (wire (pts (xy 186.69 50.8) (xy 191.77 50.8))
     (stroke (width 0) (type default) (color 0 0 0 0))
   )
@@
   )
   (wire (pts (xy 125.73 101.6) (xy 125.73 125.73))
+    (stroke (width 0) (type default) (color 0 0 0 0))
+  )
+  (wire (pts (xy 191.77 45.72) (xy 194.31 45.72))
     (stroke (width 0) (type default) (color 0 0 0 0))
   )
@@
     (stroke (width 0) (type default) (color 0 0 0 0))
   )
+  (wire (pts (xy 191.77 50.8) (xy 191.77 45.72))
+    (stroke (width 0) (type default) (color 0 0 0 0))
+  )
