File: Annahs_clock_hps/Annahs_clock_hps-backups/Annahs_clock_hps-2022-06-10_130227/Annahs_clock_hps.kicad_sch (KiCad schematic)
At the start: 11 parts, among them SW1 Omron_B3F_SPST, SW2 Omron_B3F_SPST, SW3 Omron_B3F_SPST, SW4 Omron_B3F_SPST, U1 DS1307_DIP-8, U2 MAX7219

Commit message: Update_Schematic
Parts:
- removed DS2: LED_Display_1001, footprints:Adafruit-1001-0-0-MFG, symbol HPS:LED_Display_1001
- added BT?: Battery_Cell, footprints:BatteryHolder_Keystone_106_1x20mm, symbol HPS:Battery_Cell
- added C2, C3, C7, C?: C_0805_0.1uf, footprints:C_0805_2012Metric, symbol HPS:C_0805_0.1uf
- added C4, C5: C_0805_22pf, footprints:C_0805_2012Metric, symbol HPS:C_0805_22pf
- added C6: C_0805_1uf, footprints:C_0805_2012Metric, symbol HPS:C_0805_1uf
- added C?: C_0805_10uf, footprints:C_0805_2012Metric, symbol HPS:C_0805_10uf
- added J1: Conn_01x06, footprints:PinHeader_1x06_P2.54mm_Vertical, symbol HPS:Conn_01x06
- added J2: PJ-102AH, footprints:PJ-102AH, symbol HPS:PJ-102AH
- added R3, R4, R6, R7: R_0805_4.7K, footprints:R_0805_2012Metric, symbol HPS:R_0805_4.7K
- added R5, R? (x4): R_0805_10K, footprints:R_0805_2012Metric, symbol HPS:R_0805_10K
- added R?: R_0805_22K, footprints:R_0805_2012Metric, symbol HPS:R_0805_22K
- added R? (x2): R_0805_47, footprints:R_0805_2012Metric, symbol HPS:R_0805_47
- added SW5: Omron_B3F_SPST, footprints:SW_SPST_Omron_B3FS-100xP, symbol HPS:Omron_B3F_SPST
- added U3: L7805, symbol HPS_2:L7805
- added U? (x2): SC56-11EWA, Display_7Segment:Sx56-1xxxxx, symbol HPS:SC56-11EWA
- added Y1: Crystal_16MHz, footprints:Crystal_SMD_HC49-SD, symbol HPS:Crystal_16MHz
Connections:
- net GND: now also DS1.1 (VSS), DS1.5 (R/W), BT?.2 (-), C2.2, C4.1, C5.2, C6.2, C7.2, C?.2, C?.2, J1.1 (Pin_1), J1.2 (Pin_2), J2.2 (OUT), R?.2, R?.2, R?.2, R?.2, R?.2, SW5.1 (A), SW5.2 (A), U3.2 (GND); no longer SW1.2 (A), SW2.2 (A), SW3.2 (A), SW4.2 (A)
- net VCC: now also DS1.2 (VDD), C7.1, C?.1, C?.1, R5.2, R?.2, R?.2, U3.3 (OUT); no longer SW1.4 (B), SW2.4 (B), SW3.4 (B), SW4.4 (B)
- net at U1.3 (VBAT): now also BT?.1 (+)
- net at U1.5 (SDA): now also R6.2; no longer UI1.27 (PC4)
- net at U1.6 (SCL): now also R7.2; no longer UI1.28 (PC5)
- net at U2.21 (SEG_E): now also U?.1 (E), U?.1 (E)
- net at U2.15 (SEG_F): now also U?.9 (F), U?.9 (F)
- net at U2.14 (SEG_A): now also U?.7 (A), U?.7 (A)
- net at U2.11 (DIG_1): now also U?.3 (CC), U?.8 (CC)
- net at U2.23 (SEG_D): now also U?.2 (D), U?.2 (D)
- net at U2.22 (SEG_DP): now also U?.5 (DP), U?.5 (DP)
- net at U2.20 (SEG_C): now also U?.4 (C), U?.4 (C)
- net at U2.17 (SEG_G): now also U?.10 (G), U?.10 (G)
- net at U2.16 (SEG_B): now also U?.6 (B), U?.6 (B)
- net at U2.18 (ISET): now also R?.1
- net at U2.2 (DIG_0): now also U?.3 (CC), U?.8 (CC)
- net at DS1.15 (LED(+)): now also R?.1
- net at DS1.16 (LED(-)): now also R?.1
- net at DS1.4 (RS): now also UI1.23 (PC0); no longer UI1.2 (PD0)
- net at DS1.6 (E): now also UI1.24 (PC1); no longer UI1.3 (PD1)
- net RESET: now reaches UI1.1 (~{RESET}/PC6)
- net RESET: now also R5.1
- net at UI1.10 (XTAL2/PB7): now also C5.1, Y1.1
- net at UI1.21 (AREF): now also C2.1
- net at UI1.9 (XTAL1/PB6): now also C4.2, Y1.2
- new net: R?.1, SW2.4 (B)
- new net: J1.5 (Pin_5), R4.2
- new net: R?.1, SW3.4 (B)
- new net: R?.1, SW1.4 (B)
- new net: J1.4 (Pin_4), R3.1
- new net: C3.2, J1.6 (Pin_6)
- new net: R?.1, SW4.4 (B)
- new net: C6.1, J2.1 (POLE), U3.1 (IN)
- new net: R7.1, UI1.28 (PC5)
- new net: R6.1, UI1.27 (PC4)
- new net RXD: R4.1, UI1.2 (PD0)
- new net TXD: R3.2, UI1.3 (PD1)
- new net ~{RESET}: C3.1, SW5.3 (B), SW5.4 (B)
- no-connect marks 4 -> 10
Other:
- note added: "Power Input"
- note added: "Serial"
- moved on the sheet: BZ1, C1, DS1, SW1, SW2, SW3, SW4, U1, U2, UI1

Commit message: Updated_Schematic
Parts:
- removed R? (x2): R_0805_47, footprints:R_0805_2012Metric, symbol HPS:R_0805_47
- added D?: LED_0805, footprints:LED_0805_2012Metric, symbol HPS:LED_0805
- added R?: R_0805_2.2K, footprints:R_0805_2012Metric, symbol HPS:R_0805_2.2K
- added RV1: R_POT_10K, footprints:Potentiometer_Bourns_3386P_Vertical, symbol HPS:R_POT_10K
- gave numbers to parts that had none: 10
Connections:
- net GND: now also R?.2
- net Up_SW: now reaches SW3.1 (A), UI1.6 (PD4)
- net Alarm_SW: now reaches SW1.1 (A), UI1.4 (PD2)
- net Select_SW: now reaches SW4.1 (A), UI1.11 (PD5)
- net Driver_Din: now reaches U2.1 (DIN), UI1.17 (PB3)
- net Dig0_Com: now reaches U2.11 (DIG_1), U5.3 (CC), U5.8 (CC)
- net Driver_Load: now reaches U2.12 (LOAD), UI1.16 (PB2)
- net Driver_Clk: now reaches U2.13 (CLK), UI1.19 (PB5)
- net Dig01_A: now reaches U2.14 (SEG_A), U4.7 (A), U5.7 (A)
- net Dig01_F: now reaches U2.15 (SEG_F), U4.9 (F), U5.9 (F)
- net Dig01_B: now reaches U2.16 (SEG_B), U4.6 (B), U5.6 (B)
- net Dig01_G: now reaches U2.17 (SEG_G), U4.10 (G), U5.10 (G)
- net Dig1_Com: now reaches U2.2 (DIG_0), U4.3 (CC), U4.8 (CC)
- net Dig01_C: now reaches U2.20 (SEG_C), U4.4 (C), U5.4 (C)
- net Dig01_E: now reaches U2.21 (SEG_E), U4.1 (E), U5.1 (E)
- net Dig01_DP: now reaches U2.22 (SEG_DP), U4.5 (DP), U5.5 (DP)
- net Dig01_D: now reaches U2.23 (SEG_D), U4.2 (D), U5.2 (D)
- net RTC_SCL: now reaches R7.1, UI1.28 (PC5)
- net Clk_Crystal2: now reaches C5.1, UI1.10 (XTAL2/PB7), Y1.1
- net Clk_Crystal1: now reaches C4.2, UI1.9 (XTAL1/PB6), Y1.2
- net RTC_SDA: now reaches R6.1, UI1.27 (PC4)
- net at DS1.16 (LED(-)): now also RV1.3
- net LCD_Data4: now reaches DS1.11 (D4), UI1.12 (PD6)
- net LCD_Data5: now reaches DS1.12 (D5), UI1.13 (PD7)
- net LCD_Data6: now reaches DS1.13 (D6), UI1.14 (PB0)
- net LCD_Data7: now reaches DS1.14 (D7), UI1.15 (PB1)
- net at DS1.15 (LED(+)): now also RV1.1
- net at DS1.3 (VO): now also RV1.2
- net LCD_RS: now reaches DS1.4 (RS), UI1.23 (PC0)
- net LCD_Enable: now reaches DS1.6 (E), UI1.24 (PC1)
- net Down_SW: now reaches SW2.1 (A), UI1.5 (PD3)
- net Buzzer: now reaches BZ1.1 (-), UI1.18 (PB4)
- net LED_SCK: now reaches UI1.25 (PC2)
- net LED_SCK: now also D?.2 (A)
- new net: D?.1 (K), R?.1
Other:
- note added: "LED"
- note added: "Vf = 2v Vr = 3v 10mcd @ 1.35mA therefore R=2.2KOhm"
- moved on the sheet: U4, U5

Commit message: Schematic Update
Parts:
- removed SW1, SW2, SW3, SW4: Omron_B3F_SPST, footprints:SW_SPST_Omron_B3FS-100xP, symbol HPS_3:Omron_B3F_SPST
- removed U3: L7805, symbol HPS_2:L7805
- added SW1, SW2, SW3, SW4: Omron_B3F_SPST, footprints:SW_SPST_Omron_B3FS-100xP, symbol HPS:Omron_B3F_SPST
- added U3: L7805, symbol HPS:L7805
- gave numbers to parts that had none: 2
Connections:
- net Alarm_SW: now also SW4.1 (A)
- net Down_SW: now also SW2.1 (A)
- net GND: now also U3.2 (GND)
- net Select_SW: now also SW1.1 (A)
- net Up_SW: now also SW3.1 (A)
- net VCC: now also U3.3 (OUT)
- net at R1.1: now also SW2.4 (B)
- net at R8.1: now also SW3.4 (B)
- net at R9.1: now also SW4.4 (B)
- net at R2.1: now also SW1.4 (B)
- net at C6.1, J2.1 (POLE): now also U3.1 (IN)
- no-connect marks 10 -> 25

Commit message: Schematic Update
Parts:
- removed J2: PJ-102AH, footprints:PJ-102AH, symbol HPS:PJ-102AH
- added J2: Power_inlet_vertical, footprints:Wurth-694106402002, symbol HPS:Power_inlet_vertical
Connections:
- net GND: now also J2.2 (OUT)
- net at C6.1, U3.1 (IN): now also J2.1 (POLE)
Changed lines of the file:
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@@
     (pin "1")
-  )
-  (symbol (lib_id "HPS:PJ-102AH") (at 195.58 256.54 0) (unit 1)
-    (in_bom yes) (on_board yes) (fields_autoplaced)
-    (property "Reference" "J2" (id 0) (at 193.04 243.84 0)
-      (effects (font (size 1.524 1.524)))
-    )
-    (property "Value" "PJ-102AH" (id 1) (at 193.04 247.65 0)
-      (effects (font (size 1.524 1.524)))
-    )
-    (property "Footprint" "footprints:PJ-102AH" (id 2) (at 193.04 251.46 0)
-      (effects (font (size 1.524 1.524)))
-    )
-    (property "Datasheet" "https://www.cuidevices.com/product/resource/pj-102ah.pdf" (id 3) (at 197.104 268.478 0)
-      (effects (font (size 1.524 1.524)) hide)
-    )
-    (property "MFG" "CUI Devices" (id 4) (at 195.58 274.32 0)
-      (effects (font (size 1.27 1.27)) hide)
-    )
-    (property "MPN" "PJ-102AH" (id 5) (at 195.58 276.86 0)
-      (effects (font (size 1.27 1.27)) hide)
-    )
-    (property "Digikey PN" "CP-102AH-ND" (id 6) (at 197.104 282.067 0)
-      (effects (font (size 1.27 1.27)) hide)
-    )
-    (property "Mouser PN" "490-PJ-102AH" (id 7) (at 195.58 279.273 0)
-      (effects (font (size 1.27 1.27)) hide)
-    )
-    (pin "1")
-    (pin "2")
-    (pin "3")
   )
   (symbol (lib_id "HPS:GND") (at 270.51 146.05 0) (unit 1)
@@
     (pin "2")
   )
+  (symbol (lib_id "HPS:Power_inlet_vertical") (at 195.58 256.54 0) (unit 1)
+    (in_bom yes) (on_board yes)
+    (property "Reference" "J2" (id 0) (at 193.04 243.84 0)
+      (effects (font (size 1.524 1.524)))
+    )
+    (property "Value" "Power_inlet_vertical" (id 1) (at 193.04 247.65 0)
+      (effects (font (size 1.524 1.524)))
+    )
+    (property "Footprint" "footprints:Wurth-694106402002" (id 2) (at 198.12 250.19 0)
+      (effects (font (size 1.524 1.524)))
+    )
+    (property "Datasheet" "https://www.we-online.com/katalog/datasheet/6941xx402002.pdf" (id 3) (at 197.104 268.478 0)
+      (effects (font (size 1.524 1.524)) hide)
+    )
+    (property "MFG" "Wurth" (id 4) (at 195.58 274.32 0)
+      (effects (font (size 1.27 1.27)) hide)
+    )
+    (property "MPN" "694106402002" (id 5) (at 195.58 276.86 0)
+      (effects (font (size 1.27 1.27)) hide)
+    )
+    (property "Digikey PN" "732-5931-ND" (id 6) (at 197.104 282.067 0)
+      (effects (font (size 1.27 1.27)) hide)
+    )
+    (pin "1")
+    (pin "2")
+    (pin "3")
+  )
   (symbol (lib_id "HPS:Buzzer") (at 189.23 111.76 0) (unit 1)
     (in_bom yes) (on_board yes) (fields_autoplaced)
@@
       (reference "J1") (unit 1) (value "Conn_01x06") (footprint "footprints:PinHeader_1x06_P2.54mm_Vertical")
     )
-    (path "/63eef421-fe3b-463c-a66d-6a1abae8329a"
-      (reference "J2") (unit 1) (value "PJ-102AH") (footprint "footprints:PJ-102AH")
+    (path "/f2393e9d-3944-42e3-a465-3a363f1f67da"
+      (reference "J2") (unit 1) (value "Power_inlet_vertical") (footprint "footprints:Wurth-694106402002")
     )
     (path "/0d2c0b46-b0b7-4ad3-a493-e935cfe55476"
@@
       (reference "U2") (unit 1) (value "MAX7219") (footprint "footprints:DIP-24_W7.62mm")
     )
-    (path "/13d4e30d-2d77-4560-9d16-f4925b5cccfc"
-      (reference "U3") (unit 1) (value "L7805") (footprint "")
+    (path "/19616ff1-44c3-4e50-867a-38c1b926dafa"
+      (reference "U3") (unit 1) (value "L7805") (footprint "footprints:TO-220-3_Vertical")
     )
     (path "/dd7cb9b2-3110-42e3-969d-26385b4e1f12"

Commit message: Displays_firmware
Parts:
- removed R10: R_0805_22K, footprints:R_0805_2012Metric, symbol HPS:R_0805_22K
- added R?: R_0805_100K, footprints:R_0805_2012Metric, symbol HPS:R_0805_100K
- U3: footprint (none) -> footprints:TO-220-3_Vertical
Connections:
- net VCC: now also R?.1
- net at U2.18 (ISET): now also R?.2
Other:
- moved on the sheet: C8, C9

Commit message: Clock Schematic and PCB
Parts:
- added H1, H2, H3, H4: MountingHole, footprints:MountingHole_3.2mm_M3, symbol HPS:MountingHole
- added Y2: Crystal_32768Hz, footprints:Crystal_SMD_2Pin_3.2x1.5mm, symbol HPS:Crystal_32768Hz
- gave numbers to parts that had none: 1
Connections:
- net Alarm_SW: now also R8.1, SW3.3 (B), SW3.4 (B); no longer SW4.1 (A)
- net Down_SW: now also R1.1, SW2.3 (B), SW2.4 (B); no longer SW2.1 (A)
- net GND: now also BT1.1 (+), SW1.1 (A), SW1.2 (A), SW2.1 (A), SW2.2 (A), SW3.1 (A), SW3.2 (A), SW4.1 (A), SW4.2 (A); no longer BT1.2 (-), R1.2, R2.2, R8.2, R9.2
- net Select_SW: now also R2.1, SW1.3 (B), SW1.4 (B); no longer SW1.1 (A)
- net Up_SW: now also R9.1, SW4.3 (B), SW4.4 (B); no longer SW3.1 (A)
- net VCC: now also R1.2, R2.2, R8.2, R9.2
- net VBAT: now reaches U1.3 (VBAT)
- net VBAT: now also BT1.2 (-); no longer BT1.1 (+)
- net RTC_XTAL1: now reaches U1.1 (X1)
- net RTC_XTAL1: now also Y2.1
- net RTC_XTAL2: now reaches U1.2 (X2)
- net RTC_XTAL2: now also Y2.2
- net AREF: now reaches C2.1, UI1.21 (AREF)
- no-connect marks 25 -> 15
Other:
- note added: "Bot Clock"
- note added: "Mechanical"
- moved on the sheet: BT1, C2, R1, SW2, U1

Commit message: Updated Schematic and PCB
Parts:
- removed R3, R4: R_0805_4.7K, footprints:R_0805_2012Metric, symbol HPS:R_0805_4.7K
- added R3, R4: R_0805_47, footprints:R_0805_2012Metric, symbol HPS:R_0805_47
- U4, U5: footprint Display_7Segment:Sx56-1xxxxx -> footprints:Sx56-1xxxxx
Connections:
- net GND: now also BT1.2 (-); no longer BT1.1 (+)
- net RXD: now also R4.1
- net TXD: now also R3.1
- net VBAT: now also BT1.1 (+); no longer BT1.2 (-)
- net at J1.5 (Pin_5): now also R4.2
- net at J1.4 (Pin_4): now also R3.2
Other:
- moved on the sheet: BT1
