File: Annahs_clock_hps/Annahs_clock_hps-backups/Annahs_clock_hps-2022-06-10_130227/Annahs_clock_hps.kicad_pcb (KiCad board)
At the start: 2 copper layers, 140 x 90 mm, 4 parts

Commit message: Clock Schematic
Parts:
- added BZ1: Buzzer, footprints:Buzzer_TDK_PS1240P02BT_D12.2mm_H6.5mm, F.Cu at (127.0, 119.4)
- added C1: C_0805_0.1uf, footprints:C_0805_2012Metric, F.Cu at (102.9, 137.3)
- added DS1: TC1602A-01T, footprints:TC1602A-01T, F.Cu at (109.4, 64.4)
- added DS2: LED_Display_1001, footprints:Adafruit-1001-0-0-MFG, F.Cu at (193.2, 86.7)
- added SW1: Omron_B3F_SPST, footprints:SW_SPST_Omron_B3FS-100xP, F.Cu at (138.9, 102.6)
- added SW2: Omron_B3F_SPST, footprints:SW_SPST_Omron_B3FS-100xP, F.Cu at (150.1, 102.6)
- added SW3: Omron_B3F_SPST, footprints:SW_SPST_Omron_B3FS-100xP, F.Cu at (117.2, 134.7)
- added SW4: Omron_B3F_SPST, footprints:SW_SPST_Omron_B3FS-100xP, F.Cu at (209.1, 64.8)
- added U1: DS1307_DIP-8, footprints:DIP-8_W7.62mm, F.Cu at (124.0, 100.8)
- added U2: MAX7219, footprints:DIP-24_W7.62mm, F.Cu at (113.1, 100.8)
- added UI1: ATmega328-PU, footprints:DIP-28_W7.62mm, F.Cu at (102.3, 100.8)
