File: Annahs_clock_hps/Annahs_clock_hps-backups/Annahs_clock_hps-2022-06-10_130227/Annahs_clock_hps.kicad_pcb (KiCad board)
At the start: 2 copper layers, 140 x 90 mm, 15 parts, among them SW1 Omron_B3F_SPST, SW2 Omron_B3F_SPST, SW3 Omron_B3F_SPST, SW4 Omron_B3F_SPST, U1 DS1307_DIP-8, U2 MAX7219

Commit message: Update_Schematic
Parts:
- moved DS1 1.74 mm to (107.7, 64.4)
Changed lines of the file:
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@@
   )
   (footprint "footprints:TC1602A-01T" (layer "F.Cu")
-    (at 109.441569 64.415)
+    (at 107.7 64.415)
     (descr "https://cdn-shop.adafruit.com/datasheets/TC1602A-01T.pdf")
     (tags "LCD 16x2 Alphanumeric 16pin")
@@
     (fp_arc (start 0.20066 22.9997) (mid -0.153162 22.853142) (end -0.29972 22.49932) (layer "F.SilkS") (width 0.12))
     (fp_arc (start 63.7 8) (mid 64.053553 8.146447) (end 64.2 8.5) (layer "F.SilkS") (width 0.12))
-    (fp_arc (start 64.20104 22.49932) (mid 64.054482 22.853142) (end 63.70066 22.9997) (layer "F.SilkS") (width 0.12))
+    (fp_arc (start 64.20104 22.49932) (mid 64.054473 22.853115) (end 63.70066 22.9997) (layer "F.SilkS") (width 0.12))
     (fp_line (start 72.25 -2.75) (end 72.25 33.75) (layer "F.CrtYd") (width 0.05))
     (fp_line (start -8.25 -2.75) (end 72.25 -2.75) (layer "F.CrtYd") (width 0.05))

Commit message: Updated Schematic and PCB
Parts:
- removed DS2: LED_Display_1001, footprints:Adafruit-1001-0-0-MFG
- added BT1: Battery_Cell, footprints:BatteryHolder_Keystone_106_1x20mm, F.Cu at (90.0, 73.7)
- added C2: C_0805_0.1uf, footprints:C_0805_2012Metric, F.Cu at (198.1, 106.7)
- added C3: C_0805_0.1uf, footprints:C_0805_2012Metric, F.Cu at (132.1, 88.9)
- added C4: C_0805_22pf, footprints:C_0805_2012Metric, F.Cu at (142.2, 137.2)
- added C5: C_0805_22pf, footprints:C_0805_2012Metric, F.Cu at (198.1, 96.5)
- added C6: C_0805_1uf, footprints:C_0805_2012Metric, F.Cu at (200.7, 129.5)
- added C7: C_0805_0.1uf, footprints:C_0805_2012Metric, F.Cu at (185.4, 71.1)
- added C8: C_0805_0.1uf, footprints:C_0805_2012Metric, F.Cu at (185.4, 81.3)
- added C9: C_0805_10uf, footprints:C_0805_2012Metric, F.Cu at (88.9, 129.5)
- added D1: LED_0805, footprints:LED_0805_2012Metric, F.Cu at (162.6, 88.9)
- added J1: Conn_01x06, footprints:PinHeader_1x06_P2.54mm_Vertical, F.Cu at (104.1, 92.7)
- added J2: Power_inlet_vertical, footprints:Wurth-694106402002, F.Cu at (101.6, 132.1)
- added R1: R_0805_10K, footprints:R_0805_2012Metric, F.Cu at (199.0, 114.3)
- added R10: R_0805_100K, footprints:R_0805_2012Metric, F.Cu at (121.9, 88.9)
- added R11: R_0805_2.2K, footprints:R_0805_2012Metric, F.Cu at (149.9, 88.9)
- added R2: R_0805_10K, footprints:R_0805_2012Metric, F.Cu at (199.8, 121.9)
- added R3: R_0805_4.7K, footprints:R_0805_2012Metric, F.Cu at (177.8, 86.4)
- added R4: R_0805_4.7K, footprints:R_0805_2012Metric, F.Cu at (142.2, 88.9)
- added R5: R_0805_10K, footprints:R_0805_2012Metric, F.Cu at (185.4, 63.5)
- added R6: R_0805_4.7K, footprints:R_0805_2012Metric, F.Cu at (198.1, 91.4)
- added R7: R_0805_4.7K, footprints:R_0805_2012Metric, F.Cu at (208.3, 66.0)
- added R8: R_0805_10K, footprints:R_0805_2012Metric, F.Cu at (208.3, 111.8)
- added R9: R_0805_10K, footprints:R_0805_2012Metric, F.Cu at (213.4, 127.0)
- added RV1: R_POT_10K, footprints:Potentiometer_Bourns_3386P_Vertical, F.Cu at (208.3, 121.9)
- added SW5: Omron_B3F_SPST, footprints:SW_SPST_Omron_B3FS-100xP, F.Cu at (200.7, 137.2)
- added U3: L7805, footprints:TO-220-3_Vertical, F.Cu at (114.3, 137.2)
- added U4: SC56-11EWA, footprints:Sx56-1xxxxx, F.Cu at (165.2, 78.6)
- added U5: SC56-11EWA, footprints:Sx56-1xxxxx, F.Cu at (127.1, 78.6)
- added Y1: Crystal_16MHz, footprints:Crystal_SMD_HC49-SD, F.Cu at (131.2, 137.2)
- added Y2: Crystal_32768Hz, footprints:Crystal_SMD_2Pin_3.2x1.5mm, F.Cu at (185.4, 88.9)
- moved UI1 106.1 mm to (204.5, 72.4)
- moved C1 105.5 mm to (208.3, 132.1)
- moved BZ1 84.9 mm to (193.0, 66.0)
- moved SW4 75.4 mm to (188.0, 137.2)
- moved U1 69.3 mm to (189.2, 77.4)
- moved SW3 58.1 mm to (175.3, 137.2)
- moved SW2 36.7 mm to (162.6, 137.2)
- moved SW1 36.3 mm to (149.9, 137.2)
- moved DS1 33.6 mm to (117.9, 96.4)
- moved U2 26.1 mm to (87.6, 95.2)
Connections:
- net Net-(BZ1-Pad1) renamed /Buzzer
- net Net-(DS1-Pad11) renamed /LCD_Data4
- net Net-(DS1-Pad12) renamed /LCD_Data5
- net Net-(DS1-Pad13) renamed /LCD_Data6
- net Net-(DS1-Pad14) renamed /LCD_Data7
- net Net-(U2-Pad1) renamed /Driver_Din
- net Net-(U2-Pad12) renamed /Driver_Load
- net Net-(U2-Pad13) renamed /Driver_Clk
- DS1 pad 1: unconnected-(DS1-Pad1) -> GND
- DS1 pad 15: unconnected-(DS1-Pad15) -> Net-(DS1-Pad15)
- DS1 pad 16: unconnected-(DS1-Pad16) -> Net-(DS1-Pad16)
- DS1 pad 2: unconnected-(DS1-Pad2) -> VCC
- DS1 pad 3: unconnected-(DS1-Pad3) -> Net-(DS1-Pad3)
- DS1 pad 4: Net-(DS1-Pad4) -> /LCD_RS
- DS1 pad 5: unconnected-(DS1-Pad5) -> GND
- DS1 pad 6: Net-(DS1-Pad6) -> /LCD_Enable
- SW1 pad 1: Net-(SW1-Pad1) -> GND
- SW1 pad 3: unconnected-(SW1-Pad3) -> /Select_SW
- SW1 pad 4: VCC -> /Select_SW
- SW2 pad 1: Net-(SW2-Pad1) -> GND
- SW2 pad 3: unconnected-(SW2-Pad3) -> /Down_SW
- SW2 pad 4: VCC -> /Down_SW
- SW3 pad 1: Net-(SW3-Pad1) -> GND
- SW3 pad 3: unconnected-(SW3-Pad3) -> /Alarm_SW
- SW3 pad 4: VCC -> /Alarm_SW
- SW4 pad 1: Net-(SW4-Pad1) -> GND
- SW4 pad 3: unconnected-(SW4-Pad3) -> /Up_SW
- SW4 pad 4: VCC -> /Up_SW
- U1 pad 1: unconnected-(U1-Pad1) -> /RTC_XTAL1
- U1 pad 2: unconnected-(U1-Pad2) -> /RTC_XTAL2
- U1 pad 3: unconnected-(U1-Pad3) -> /VBAT
- U1 pad 5: Net-(U1-Pad5) -> Net-(R6-Pad2)
- U1 pad 6: Net-(U1-Pad6) -> Net-(R7-Pad2)
- U2 pad 11: Net-(DS2-Pad14) -> /Dig0_Com
- U2 pad 14: Net-(DS2-Pad13) -> /Dig01_A
- U2 pad 15: Net-(DS2-Pad12) -> /Dig01_F
- U2 pad 16: Net-(DS2-Pad9) -> /Dig01_B
- U2 pad 17: Net-(DS2-Pad5) -> /Dig01_G
- U2 pad 18: unconnected-(U2-Pad18) -> Net-(R10-Pad2)
- U2 pad 2: unconnected-(U2-Pad2) -> /Dig1_Com
- U2 pad 20: Net-(DS2-Pad4) -> /Dig01_C
- U2 pad 21: Net-(DS2-Pad1) -> /Dig01_E
- U2 pad 22: Net-(DS2-Pad3) -> /Dig01_DP
- U2 pad 23: Net-(DS2-Pad2) -> /Dig01_D
- UI1 pad 1: unconnected-(UI1-Pad1) -> RESET
- UI1 pad 10: unconnected-(UI1-Pad10) -> /Clk_Crystal2
- UI1 pad 11: Net-(SW4-Pad1) -> /Select_SW
- UI1 pad 2: Net-(DS1-Pad4) -> RXD
- UI1 pad 21: unconnected-(UI1-Pad21) -> /AREF
- UI1 pad 23: unconnected-(UI1-Pad23) -> /LCD_RS
- UI1 pad 24: unconnected-(UI1-Pad24) -> /LCD_Enable
- UI1 pad 25: unconnected-(UI1-Pad25) -> LED_SCK
- UI1 pad 27: Net-(U1-Pad5) -> /RTC_SDA
- UI1 pad 28: Net-(U1-Pad6) -> /RTC_SCL
- UI1 pad 3: Net-(DS1-Pad6) -> TXD
- UI1 pad 4: Net-(SW1-Pad1) -> /Alarm_SW
- UI1 pad 5: Net-(SW2-Pad1) -> /Down_SW
- UI1 pad 6: Net-(SW3-Pad1) -> /Up_SW
- UI1 pad 9: unconnected-(UI1-Pad9) -> /Clk_Crystal1
