File: Annahs_clock_hps/Annahs_clock_hps-backups/Annahs_clock_hps-2022-06-10_130227/_autosave-Annahs_clock_hps.kicad_sch (KiCad schematic)
At the start: 11 parts, among them SW1 Omron_B3F_SPST, SW2 Omron_B3F_SPST, SW3 Omron_B3F_SPST, SW4 Omron_B3F_SPST, U1 DS1307_DIP-8, U2 MAX7219

Commit message: Clock Schematic
Parts:
- added C? (x3): C_0805_0.1uf, footprints:C_0805_2012Metric, symbol HPS:C_0805_0.1uf
- added C?: C_0805_1uf, footprints:C_0805_2012Metric, symbol HPS:C_0805_1uf
- added J?: PJ-102AH, footprints:PJ-102AH, symbol HPS:PJ-102AH
- added J?: Conn_01x06, footprints:PinHeader_1x06_P2.54mm_Vertical, symbol HPS:Conn_01x06
- added R1, R2: R_0805_1K, footprints:R_0805_2012Metric, symbol HPS:R_0805_1K
- added R? (x2): R_0805_4.7K, footprints:R_0805_2012Metric, symbol HPS:R_0805_4.7K
- added R?: R_0805_10K, footprints:R_0805_2012Metric, symbol HPS:R_0805_10K
- added SW?: Omron_B3F_SPST, footprints:SW_SPST_Omron_B3FS-100xP, symbol HPS:Omron_B3F_SPST
- added U?: L7805, symbol HPS_2:L7805
Connections:
- net GND: now also DS1.1 (VSS), DS1.5 (R/W), SW1.4 (B), SW2.4 (B), SW3.4 (B), SW4.4 (B), U1.3 (VBAT), C?.2, C?.2, C?.2, J?.1 (Pin_1), J?.2 (OUT), J?.2 (Pin_2), R2.2, SW?.1 (A), SW?.2 (A), U?.2 (GND); no longer SW1.2 (A), SW2.2 (A), SW3.2 (A), SW4.2 (A)
- net VCC: now also DS1.2 (VDD), C?.1, R1.2, U?.3 (OUT); no longer SW1.4 (B), SW2.4 (B), SW3.4 (B), SW4.4 (B)
- net at DS2.14 (COM_DIG.1): now also U2.2 (DIG_0); no longer U2.11 (DIG_1)
- net at DS1.15 (LED(+)): now also R1.1
- net at DS1.16 (LED(-)): now also R2.1
- net at DS1.4 (RS): now also UI1.23 (PC0); no longer UI1.2 (PD0)
- net at DS1.6 (E): now also UI1.24 (PC1); no longer UI1.3 (PD1)
- net at UI1.1 (~{RESET}/PC6): now also R?.1
- net at UI1.21 (AREF): now also C?.1
- new net: J?.5 (Pin_5), R?.2
- new net: J?.4 (Pin_4), R?.1
- new net: C?.2, J?.6 (Pin_6)
- new net: C?.1, J?.1 (POLE), U?.1 (IN)
- new net RXD: R?.1, UI1.2 (PD0)
- new net TXD: R?.2, UI1.3 (PD1)
- new net ~{RESET}: C?.1, SW?.3 (B), SW?.4 (B)
- no-connect marks 4 -> 9
Other:
- note added: "Power Input"
- note added: "Serial"
- moved on the sheet: BZ1, C1, DS1, DS2, SW1, SW2, SW3, SW4, U1, U2, UI1

Commit message: Update_Schematic
Parts:
- removed DS2: LED_Display_1001, footprints:Adafruit-1001-0-0-MFG, symbol HPS:LED_Display_1001
- removed R1, R2: R_0805_1K, footprints:R_0805_2012Metric, symbol HPS:R_0805_1K
- added BT1: Battery_Cell, footprints:BatteryHolder_Keystone_106_1x20mm, symbol HPS:Battery_Cell
- added C4, C5: C_0805_22pf, footprints:C_0805_2012Metric, symbol HPS:C_0805_22pf
- added C8: C_0805_0.1uf, footprints:C_0805_2012Metric, symbol HPS:C_0805_0.1uf
- added C9: C_0805_10uf, footprints:C_0805_2012Metric, symbol HPS:C_0805_10uf
- added R1, R2, R8, R9: R_0805_10K, footprints:R_0805_2012Metric, symbol HPS:R_0805_10K
- added R10: R_0805_22K, footprints:R_0805_2012Metric, symbol HPS:R_0805_22K
- added R6, R7: R_0805_4.7K, footprints:R_0805_2012Metric, symbol HPS:R_0805_4.7K
- added RV1: R_POT_10K, footprints:Potentiometer_Bourns_3386P_Vertical, symbol HPS:R_POT_10K
- added U4, U5: SC56-11EWA, Display_7Segment:Sx56-1xxxxx, symbol HPS:SC56-11EWA
- added Y1: Crystal_16MHz, footprints:Crystal_SMD_HC49-SD, symbol HPS:Crystal_16MHz
- gave numbers to parts that had none: 11
Connections:
- net GND: now also BT1.2 (-), C4.1, C5.2, C8.2, C9.2, R1.2, R2.2, R8.2, R9.2; no longer SW1.4 (B), SW2.4 (B), SW3.4 (B), SW4.4 (B), U1.3 (VBAT)
- net VCC: now also R5.2, C8.1, C9.1, R10.2
- net at U1.5 (SDA): now also R6.2; no longer UI1.27 (PC4)
- net at U1.6 (SCL): now also R7.2; no longer UI1.28 (PC5)
- net at U2.21 (SEG_E): now also U4.1 (E), U5.1 (E)
- net at U2.15 (SEG_F): now also U4.9 (F), U5.9 (F)
- net Dig0_A: now reaches U2.14 (SEG_A)
- net Dig0_A: now also U4.7 (A), U5.7 (A)
- net at U2.2 (DIG_0): now also U4.3 (CC), U4.8 (CC)
- net at U2.23 (SEG_D): now also U4.2 (D), U5.2 (D)
- net at U2.22 (SEG_DP): now also U4.5 (DP), U5.5 (DP)
- net at U2.20 (SEG_C): now also U4.4 (C), U5.4 (C)
- net at U2.17 (SEG_G): now also U4.10 (G), U5.10 (G)
- net Dig0_B: now reaches U2.16 (SEG_B)
- net Dig0_B: now also U4.6 (B), U5.6 (B)
- net Up_SW: now reaches SW3.1 (A), UI1.6 (PD4)
- net Alarm_SW: now reaches SW1.1 (A), UI1.4 (PD2)
- net Select_SW: now reaches SW4.1 (A), UI1.11 (PD5)
- net Driver_Din: now reaches U2.1 (DIN), UI1.17 (PB3)
- net at U2.11 (DIG_1): now also U5.3 (CC), U5.8 (CC)
- net Driver_Load: now reaches U2.12 (LOAD), UI1.16 (PB2)
- net Driver_Clk: now reaches U2.13 (CLK), UI1.19 (PB5)
- net at U2.18 (ISET): now also R10.1
- net at DS1.16 (LED(-)): now also RV1.3
- net LCD_Data4: now reaches DS1.11 (D4), UI1.12 (PD6)
- net LCD_Data5: now reaches DS1.12 (D5), UI1.13 (PD7)
- net LCD_Data6: now reaches DS1.13 (D6), UI1.14 (PB0)
- net LCD_Data7: now reaches DS1.14 (D7), UI1.15 (PB1)
- net at DS1.15 (LED(+)): now also RV1.1
- net at DS1.3 (VO): now also RV1.2
- net LCD_RS: now reaches DS1.4 (RS), UI1.23 (PC0)
- net LCD_Enable: now reaches DS1.6 (E), UI1.24 (PC1)
- net Down_SW: now reaches SW2.1 (A), UI1.5 (PD3)
- net RESET: now reaches R5.1, UI1.1 (~{RESET}/PC6)
- net Clk_Crystal2: now reaches UI1.10 (XTAL2/PB7)
- net Clk_Crystal2: now also C5.1, Y1.1
- net Buzzer: now reaches BZ1.1 (-), UI1.18 (PB4)
- net Clk_Crystal1: now reaches UI1.9 (XTAL1/PB6)
- net Clk_Crystal1: now also C4.2, Y1.2
- new net: BT1.1 (+), U1.3 (VBAT)
- new net: R1.1, SW2.4 (B)
- new net: R8.1, SW3.4 (B)
- new net: R9.1, SW1.4 (B)
- new net: R2.1, SW4.4 (B)
- new net RTC_SCL: R7.1, UI1.28 (PC5)
- new net RTC_SDA: R6.1, UI1.27 (PC4)
- no-connect marks 9 -> 10
Other:
- moved on the sheet: BZ1, C1, C2, C3, C6, C7, DS1, J1, J2, R3, R4, R5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
