File: Annahs_clock_hps/Annahs_clock_hps-backups/Annahs_clock_hps-2022-06-10_130227/Annahs_clock_hps-backups/Annahs_clock_hps-2022-06-23_181852/Annahs_clock_hps.kicad_sch (KiCad schematic)
At the start: 11 parts, among them SW1 Omron_B3F_SPST, SW2 Omron_B3F_SPST, SW3 Omron_B3F_SPST, SW4 Omron_B3F_SPST, U1 DS1307_DIP-8, U2 MAX7219

Commit message: Clock Schematic
Parts:
- removed DS2: LED_Display_1001, footprints:Adafruit-1001-0-0-MFG, symbol HPS:LED_Display_1001
Connections:
- net GND: no longer U2.4 (GND), U2.9 (GND)
- net VCC: no longer U2.19 (V+)
Other:
- moved on the sheet: BZ1, C1, DS1, SW1, SW2, SW3, SW4, U1, U2, UI1
