File: Annahs_clock_hps/Schematic and PCB/Annahs_clock_hps.kicad_sch (KiCad schematic)
At the start: 66 parts, among them J1 Conn_01x06, J2 Power_inlet_vertical, J3 Conn_02x03_Odd_Even, Q1 NPN_2N3904_SOT23, SW1 Omron_B3F_SPST, SW2 Omron_B3F_SPST, SW3 Omron_B3F_SPST, SW4 Omron_B3F_SPST, SW5 Omron_B3F_SPST, SW6 Omron_B3F_SPST, U1 DS1307_DIP-8, U2 MAX7219, U3 L7805, U4 SC56-11EWA, U5 SC56-11EWA, Y1 Crystal_16MHz, Y2 Crystal_32768Hz

Commit message: Updated Schematic and PCB
Parts:
- added H1, H2, H3, H4: MountingHole, footprints:MountingHole_3.2mm_M3, symbol HPS:MountingHole
Other:
- note added: "Mechanical"
Changed lines of the file:
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@@
   (junction (at 279.4 54.61) (diameter 0) (color 0 0 0 0)
   )
+  (junction (at 248.92 152.4) (diameter 0) (color 0 0 0 0)
+  )
   (junction (at 281.94 57.15) (diameter 0) (color 0 0 0 0)
   )
@@
     (stroke (width 0) (type default) (color 0 0 0 0))
   )
+  (polyline (pts (xy 271.78 187.96) (xy 320.04 187.96))
+    (stroke (width 0) (type default) (color 0 0 0 0))
+  )
   (wire (pts (xy 101.6 137.16) (xy 119.38 137.16))
     (stroke (width 0) (type default) (color 0 0 0 0))
@@
     (stroke (width 0) (type default) (color 0 0 0 0))
   )
-  (wire (pts (xy 252.73 152.4) (xy 245.11 152.4))
+  (wire (pts (xy 252.73 152.4) (xy 248.92 152.4))
     (stroke (width 0) (type default) (color 0 0 0 0))
   )
@@
     (stroke (width 0) (type default) (color 0 0 0 0))
   )
+  (polyline (pts (xy 271.78 212.09) (xy 320.04 212.09))
+    (stroke (width 0) (type default) (color 0 0 0 0))
+  )
   (wire (pts (xy 110.49 185.42) (xy 110.49 182.88))
     (stroke (width 0) (type default) (color 0 0 0 0))
@@
     (stroke (width 0) (type default) (color 0 0 0 0))
   )
+  (polyline (pts (xy 320.04 212.09) (xy 320.04 187.96))
+    (stroke (width 0) (type default) (color 0 0 0 0))
+  )
   (wire (pts (xy 124.46 116.84) (xy 205.74 116.84))
     (stroke (width 0) (type default) (color 0 0 0 0))
@@
     (stroke (width 0) (type default) (color 0 0 0 0))
   )
+  (wire (pts (xy 248.92 152.4) (xy 245.11 152.4))
+    (stroke (width 0) (type default) (color 0 0 0 0))
+  )
   (polyline (pts (xy 80.01 275.59) (xy 163.83 275.59))
     (stroke (width 0) (type default) (color 0 0 0 0))
@@
     (stroke (width 0) (type default) (color 0 0 0 0))
   )
+  (polyline (pts (xy 271.78 187.96) (xy 271.78 212.09))
+    (stroke (width 0) (type default) (color 0 0 0 0))
+  )
   (wire (pts (xy 290.83 44.45) (xy 290.83 64.77))
     (stroke (width 0) (type default) (color 0 0 0 0))
@@
     (effects (font (size 1.27 1.27)) (justify left bottom))
   )
+  (text "Mechanical" (at 303.53 210.82 180)
+    (effects (font (size 3 3) bold) (justify right bottom))
+  )
   (text "Power TP\n" (at 307.34 247.65 0)
     (effects (font (size 3 3) (thickness 0.6) bold) (justify left bottom))
@@
     (effects (font (size 1.27 1.27)) (justify left bottom))
   )
-  (label "Serial_RXD" (at 104.14 147.32 0)
+  (label "RXD" (at 104.14 147.32 0)
     (effects (font (size 1.27 1.27)) (justify left bottom))
   )
@@
     (effects (font (size 1.27 1.27)) (justify left bottom))
   )
-  (label "Driver_Clk" (at 102.87 116.84 0)
+  (label "LED_SCK" (at 102.87 116.84 0)
     (effects (font (size 1.27 1.27)) (justify left bottom))
   )
@@
     (effects (font (size 1.27 1.27)) (justify left bottom))
   )
-  (label "Alarm Off Button" (at 102.87 114.3 0)
+  (label "MISO" (at 102.87 114.3 0)
     (effects (font (size 1.27 1.27)) (justify left bottom))
   )
@@
     (effects (font (size 1.27 1.27)) (justify left bottom))
   )
-  (label "Serial_TXD" (at 104.14 149.86 0)
+  (label "TXD" (at 104.14 149.86 0)
     (effects (font (size 1.27 1.27)) (justify left bottom))
   )
@@
     (effects (font (size 1.27 1.27)) (justify left bottom))
   )
-  (label "Driver_Din" (at 102.87 111.76 0)
+  (label "MOSI" (at 102.87 111.76 0)
     (effects (font (size 1.27 1.27)) (justify left bottom))
   )
@@
     (pin "1")
   )
+  (symbol (lib_id "HPS:MountingHole") (at 278.13 199.39 0) (unit 1)
+    (in_bom yes) (on_board yes) (fields_autoplaced)
+    (property "Reference" "H2" (id 0) (at 280.67 198.1199 0)
+      (effects (font (size 1.27 1.27)) (justify left))
+    )
+    (property "Value" "MountingHole" (id 1) (at 280.67 200.6599 0)
+      (effects (font (size 1.27 1.27)) (justify left))
+    )
+    (property "Footprint" "footprints:MountingHole_3.2mm_M3" (id 2) (at 278.13 199.39 0)
+      (effects (font (size 1.27 1.27)) hide)
+    )
+    (property "Datasheet" "~" (id 3) (at 278.13 199.39 0)
+      (effects (font (size 1.27 1.27)) hide)
+    )
+  )
   (symbol (lib_id "HPS:TestPoint") (at 308.61 234.95 180) (unit 1)
     (in_bom yes) (on_board yes) (fields_autoplaced)
@@
     (pin "1")
   )
+  (symbol (lib_id "HPS:MountingHole") (at 278.13 191.77 0) (unit 1)
+    (in_bom yes) (on_board yes) (fields_autoplaced)
+    (property "Reference" "H1" (id 0) (at 280.67 190.4999 0)
+      (effects (font (size 1.27 1.27)) (justify left))
+    )
+    (property "Value" "MountingHole" (id 1) (at 280.67 193.0399 0)
+      (effects (font (size 1.27 1.27)) (justify left))
+    )
+    (property "Footprint" "footprints:MountingHole_3.2mm_M3" (id 2) (at 278.13 191.77 0)
+      (effects (font (size 1.27 1.27)) hide)
+    )
+    (property "Datasheet" "~" (id 3) (at 278.13 191.77 0)
+      (effects (font (size 1.27 1.27)) hide)
+    )
+  )
   (symbol (lib_id "HPS:Omron_B3F_SPST") (at 129.54 210.82 0) (unit 1)
     (in_bom yes) (on_board yes)
@@
     (pin "2")
   )
+  (symbol (lib_id "HPS:MountingHole") (at 299.72 199.39 0) (unit 1)
+    (in_bom yes) (on_board yes) (fields_autoplaced)
+    (property "Reference" "H4" (id 0) (at 302.26 198.1199 0)
+      (effects (font (size 1.27 1.27)) (justify left))
+    )
+    (property "Value" "MountingHole" (id 1) (at 302.26 200.6599 0)
+      (effects (font (size 1.27 1.27)) (justify left))
+    )
+    (property "Footprint" "footprints:MountingHole_3.2mm_M3" (id 2) (at 299.72 199.39 0)
+      (effects (font (size 1.27 1.27)) hide)
+    )
+    (property "Datasheet" "~" (id 3) (at 299.72 199.39 0)
+      (effects (font (size 1.27 1.27)) hide)
+    )
+  )
   (symbol (lib_id "HPS:C_0805_10uf") (at 227.33 69.85 90) (unit 1)
     (in_bom yes) (on_board yes)
@@
     (pin "1")
   )
+  (symbol (lib_id "HPS:PWR_FLAG") (at 248.92 152.4 0) (unit 1)
+    (in_bom yes) (on_board yes) (fields_autoplaced)
+    (property "Reference" "#FLG0101" (id 0) (at 248.92 150.495 0)
+      (effects (font (size 1.27 1.27)) hide)
+    )
+    (property "Value" "PWR_FLAG" (id 1) (at 248.92 147.32 0))
+    (property "Footprint" "" (id 2) (at 248.92 152.4 0)
+      (effects (font (size 1.27 1.27)) hide)
+    )
+    (property "Datasheet" "~" (id 3) (at 248.92 152.4 0)
+      (effects (font (size 1.27 1.27)) hide)
+    )
+    (pin "1")
+  )
   (symbol (lib_id "HPS:R_POT_10K") (at 278.13 142.24 180) (unit 1)
     (in_bom yes) (on_board yes)
@@
     (pin "2")
   )
+  (symbol (lib_id "HPS:MountingHole") (at 299.72 191.77 0) (unit 1)
+    (in_bom yes) (on_board yes) (fields_autoplaced)
+    (property "Reference" "H3" (id 0) (at 302.26 190.4999 0)
+      (effects (font (size 1.27 1.27)) (justify left))
+    )
+    (property "Value" "MountingHole" (id 1) (at 302.26 193.0399 0)
+      (effects (font (size 1.27 1.27)) (justify left))
+    )
+    (property "Footprint" "footprints:MountingHole_3.2mm_M3" (id 2) (at 299.72 191.77 0)
+      (effects (font (size 1.27 1.27)) hide)
+    )
+    (property "Datasheet" "~" (id 3) (at 299.72 191.77 0)
+      (effects (font (size 1.27 1.27)) hide)
+    )
+  )
   (symbol (lib_id "HPS:HPS_Logo") (at 382.27 260.35 0) (unit 1)
     (in_bom yes) (on_board yes) (fields_autoplaced)
@@
       (reference "#FLG04") (unit 1) (value "PWR_FLAG") (footprint "")
     )
+    (path "/ad15b4a4-7e27-4123-897c-252c0852afbc"
+      (reference "#FLG0101") (unit 1) (value "PWR_FLAG") (footprint "")
+    )
     (path "/e4ba8235-a879-4293-a3fa-90a9eab92330"
       (reference "#G1") (unit 1) (value "HPS_Logo") (footprint "")
@@
       (reference "DS1") (unit 1) (value "TC1602A-01T") (footprint "footprints:TC1602A-01T")
     )
+    (path "/7871a977-e975-42a9-8858-2166ba76271e"
+      (reference "H1") (unit 1) (value "MountingHole") (footprint "footprints:MountingHole_3.2mm_M3")
+    )
+    (path "/46a67faf-6ca9-49ff-8878-a48d4a198a70"
+      (reference "H2") (unit 1) (value "MountingHole") (footprint "footprints:MountingHole_3.2mm_M3")
+    )
+    (path "/e2c4b375-ad86-4f72-bf41-0759711039a4"
+      (reference "H3") (unit 1) (value "MountingHole") (footprint "footprints:MountingHole_3.2mm_M3")
+    )
+    (path "/833170ec-1560-4758-bb76-d2fe11b9ca0a"
+      (reference "H4") (unit 1) (value "MountingHole") (footprint "footprints:MountingHole_3.2mm_M3")
+    )
     (path "/dae78a19-1fcd-4bca-a7a8-31e810ab721c"
