File: Annahs_clock_hps/Schematic and PCB/Annahs_clock_hps.kicad_pcb (KiCad board)
At the start: 2 copper layers, 140 x 90 mm, 70 parts, among them J1 Conn_01x06, J2 Power_inlet_vertical, J3 Conn_02x03_Odd_Even, Q1 NPN_2N3904_SOT23, SW1 Omron_B3F_SPST, SW2 Omron_B3F_SPST, SW3 Omron_B3F_SPST, SW4 Omron_B3F_SPST, SW5 Omron_B3F_SPST, SW6 Omron_B3F_SPST, U1 DS1307_DIP-8, U2 MAX7219, U3 L7805, U4 SC56-11EWA, U5 SC56-11EWA, Y1 Crystal_16MHz, Y2 Crystal_32768Hz

Commit message: Updated Schematic and PCB
Parts:
- BT1: moved to B.Cu

Commit message: Updated PCB and Schematic
Parts:
- J1, J3: moved to B.Cu
- moved R5 42.9 mm to (193.0, 116.4), turned to 90 degrees
- moved C4 21.8 mm to (195.6, 94.0), turned to 180 degrees
- moved Y1 8.12 mm to (191.1, 89.5), turned to 0 degrees
- moved C1 6.14 mm to (196.2, 84.0), turned to 180 degrees
- moved C5 3.51 mm to (182.9, 90.0), turned to -90 degrees
- moved J3 2.55 mm to (215.3, 95.2), turned to 180 degrees
- turned J1 to 180 degrees
Routing:
- net ~{RESET}: track 108.4 -> 139.0 mm, vias 2 -> 6
- net /Clk_Crystal1: track 34.9 -> 10.9 mm, vias 2 -> 0
- net GND: track 196.0 -> 206.1 mm, vias 19 -> 21
- net MOSI: track 147.2 -> 139.7 mm
- net VCC: track 44.0 -> 50.0 mm, vias 1 -> 0
- net /Select_SW: track 74.8 -> 72.7 mm
- net /Clk_Crystal2: track 19.1 -> 21.1 mm, vias 2 -> 0
- net MISO: track 168.2 -> 169.8 mm
- net LED_SCK: track 176.2 -> 177.7 mm, vias 6 -> 4
- net /LCD_Data7: track 69.2 -> 70.5 mm
- net /Dig01_DP: track 84.4 -> 83.1 mm
- net /Dig0_Com: track 89.8 -> 88.7 mm
- net TXD: track 44.9 -> 45.9 mm
- net /Driver_Load: track 142.4 -> 143.3 mm
- net /Dig01_B: track 101.4 -> 100.6 mm
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
Commit message: Updated Gerber, STEP, BOM
Parts:
- added G***: LOGO, footprints:HPS_logo, B.Cu at (146.7, 120.0)
- moved C4 1.27 mm to (194.3, 94.0)
- moved C5 1.27 mm to (181.6, 90.0)
- moved Y1 1.27 mm to (189.9, 89.5)
Routing:
- net GND: track 206.1 -> 210.3 mm, vias 21 -> 20
